File: kicad/esp32-controller.kicad_sch (KiCad schematic)
At the start: 2 parts

Commit message: init
Parts:
- removed U? (x2): ~, yvolodym.switches:Joystick_PS5, symbol PCM_yvolodym:Joystick_PS5
- added U1, U2: PS4, PCM_yvolodym:Joystick_PS5, symbol PCM_yvolodym:Joystick_PS5
Other:
- added sheet supply (supply.kicad_sch)

Commit message: init
Parts:
- added U3: ESP32, PCM_yvolodym:ESP32-WROVER-B, symbol PCM_yvolodym:ESP32-WROVER-IB
Connections:
- new net: U3.1 (GND), U3.15 (GND), U3.38 (GND), U3.39 (GND)
Changed lines of the file:
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@@
 	(generator_version "9.0")
 	(paper "A4")
+	(junction
+		(at 52.07 99.06)
+		(diameter 0)
+		(color 0 0 0 0)
+	)
+	(junction
+		(at 52.07 116.84)
+		(diameter 0)
+		(color 0 0 0 0)
+	)
 	(wire
 		(pts
@@
 	(wire
 		(pts
+			(xy 72.39 132.08) (xy 72.39 127)
+		)
+		(stroke
+			(width 0)
+			(type default)
+		)
+	)
+	(wire
+		(pts
 			(xy 128.27 96.52) (xy 123.19 96.52)
 		)
@@
 	(wire
 		(pts
+			(xy 83.82 99.06) (xy 88.9 99.06)
+		)
+		(stroke
+			(width 0)
+			(type default)
+		)
+	)
+	(wire
+		(pts
+			(xy 52.07 116.84) (xy 60.96 116.84)
+		)
+		(stroke
+			(width 0)
+			(type default)
+		)
+	)
+	(wire
+		(pts
 			(xy 128.27 31.75) (xy 128.27 96.52)
 		)
@@
 	(wire
 		(pts
+			(xy 52.07 132.08) (xy 72.39 132.08)
+		)
+		(stroke
+			(width 0)
+			(type default)
+		)
+	)
+	(wire
+		(pts
+			(xy 52.07 99.06) (xy 52.07 116.84)
+		)
+		(stroke
+			(width 0)
+			(type default)
+		)
+	)
+	(wire
+		(pts
+			(xy 88.9 95.25) (xy 52.07 95.25)
+		)
+		(stroke
+			(width 0)
+			(type default)
+		)
+	)
+	(wire
+		(pts
 			(xy 121.92 26.67) (xy 132.08 26.67)
 		)
@@
 	(wire
 		(pts
+			(xy 88.9 99.06) (xy 88.9 95.25)
+		)
+		(stroke
+			(width 0)
+			(type default)
+		)
+	)
+	(wire
+		(pts
 			(xy 132.08 93.98) (xy 123.19 93.98)
 		)
@@
 	(wire
 		(pts
+			(xy 52.07 95.25) (xy 52.07 99.06)
+		)
+		(stroke
+			(width 0)
+			(type default)
+		)
+	)
+	(wire
+		(pts
+			(xy 52.07 116.84) (xy 52.07 132.08)
+		)
+		(stroke
+			(width 0)
+			(type default)
+		)
+	)
+	(wire
+		(pts
 			(xy 95.25 147.32) (xy 95.25 154.94)
 		)
@@
 		(pts
 			(xy 121.92 31.75) (xy 128.27 31.75)
+		)
+		(stroke
+			(width 0)
+			(type default)
+		)
+	)
+	(wire
+		(pts
+			(xy 60.96 99.06) (xy 52.07 99.06)
 		)
 		(stroke
@@
 					(unit 1)
 				)
+			)
+		)
+	)
+	(symbol
+		(lib_id "PCM_yvolodym:ESP32-WROVER-IB")
+		(at 72.39 95.25 0)
+		(unit 1)
+		(exclude_from_sim no)
+		(in_bom yes)
+		(on_board yes)
+		(dnp no)
+		(fields_autoplaced yes)
+		(property "Reference" "U3"
+			(at 72.39 91.44 0)
+			(effects
+				(font
+					(size 1.27 1.27)
+				)
+			)
+		)
+		(property "Value" "ESP32"
+			(at 72.39 93.98 0)
+			(effects
+				(font
+					(size 1.27 1.27)
+				)
+			)
+		)
+		(property "Footprint" "PCM_yvolodym:ESP32-WROVER-B"
+			(at 72.39 95.25 0)
+			(effects
+				(font
+					(size 1.27 1.27)
+				)
+				(hide yes)
+			)
+		)
+		(property "Datasheet" ""
+			(at 72.39 95.25 0)
+			(effects
+				(font
+					(size 1.27 1.27)
+				)
+				(hide yes)
+			)
+		)
+		(property "Description" "ESP32-WROVER-IB"
+			(at 72.39 95.25 0)
+			(effects
+				(font
+					(size 1.27 1.27)
+				)
+				(hide yes)
+			)
+		)
+		(pin "15"
+		)
+		(pin "9"
+		)
+		(pin "4"
+		)
+		(pin "19"
+		)
+		(pin "8"
+		)
+		(pin "5"
+		)
+		(pin "6"
+		)
+		(pin "12"
+		)
+		(pin "14"
+		)
+		(pin "2"
+		)
+		(pin "17"
+		)
+		(pin "18"
+		)
+		(pin "35"
+		)
+		(pin "25"
+		)
+		(pin "13"
+		)
+		(pin "10"
+		)
+		(pin "1"
+		)
+		(pin "7"
+		)
+		(pin "11"
+		)
+		(pin "3"
+		)
+		(pin "16"
+		)
+		(pin "39"
+		)
+		(pin "38"
+		)
+		(pin "37"
+		)
+		(pin "36"
+		)
+		(pin "34"
+		)
+		(pin "33"
+		)
+		(pin "31"
+		)
+		(pin "30"
+		)
+		(pin "29"
+		)
+		(pin "26"
+		)
+		(pin "21"
+		)
+		(pin "20"
+		)
+		(pin "22"
+		)
+		(pin "23"
+		)
+		(pin "24"
+		)
+		(instances
+			(project ""
+				(path "/1b61a099-fa01-45c5-bfa6-c1f023697108"
+					(reference "U3")
+					(unit 1)
+				)

Commit message: init
Parts:
- added C1, C2: 100nF, Capacitor_SMD:C_1206_3216Metric, symbol Device:C
- added D1, D2: YELLOW, Diode_SMD:D_0603_1608Metric, symbol Device:LED
- added J1: Conn_01x08_Socket, Connector_PinSocket_2.54mm:PinSocket_1x08_P2.54mm_Vertical, symbol Connector:Conn_01x08_Pin
- added Q1, Q2: BCW66G, Package_TO_SOT_SMD:SOT-23, symbol Simulation_SPICE:NPN
- added R1, R2: 2K, Resistor_SMD:R_1206_3216Metric, symbol Device:R
- added R3, R4, R5, R6, R7: 10K, Resistor_SMD:R_1206_3216Metric, symbol Device:R
- added R8, R9: 470, Resistor_SMD:R_1206_3216Metric, symbol Device:R
- added SW1, SW2: RESET, Button_Switch_SMD:SW_Push_1P1T_NO_CK_KMR2, symbol Switch:CK_KMS2xxG
- added U4: CH340C, Package_SO:SOIC-16_3.9x9.9mm_P1.27mm, symbol Interface_USB:CH340C
- U1: renamed from U3; value ESP32 -> ESP32-WROVER-IB
- renumbered U1 to U2, U2 to U3
Connections:
- net +3.3V: now also U1.2 (VDD33), J1.2 (Pin_2), R1.1, R2.1, R3.1, R4.1, R5.1, U4.16 (VCC), U4.4 (V3)
- net GND: now also U1.1 (GND), U1.15 (GND), U1.38 (GND), U1.39 (GND), U2.H1 (H+), U2.H3 (H-), U2.S1 (SHIELD), U2.S2 (SHIELD), U2.S3 (SHIELD), U2.S4 (SHIELD), U2.V1 (V+), U2.V3 (V-), U3.H1 (H+), U3.H3 (H-), U3.S1 (SHIELD), U3.S2 (SHIELD), U3.S3 (SHIELD), U3.S4 (SHIELD), U3.V1 (V+), U3.V3 (V-), C1.2, C2.2, J1.1 (Pin_1), SW1.1, SW1.SH (B), SW2.1, SW2.SH (B), U4.1 (GND)
- net supply/D+: now also U4.5 (UD+)
- net supply/D-: now also U4.6 (UD-)
- net VRy: now reaches U2.H2 (H)
- net VRy: now also U1.9 (GPIO33)
- net VRx: now reaches U2.V2 (V)
- net VRx: now also U1.8 (GPIO32)
- net at U1.12 (GPIO27): now also D1.1 (K)
- net GPIO15: now reaches U1.23 (GPIO15)
- net GPIO15: now also J1.8 (Pin_8)
- net GPIO2: now reaches U1.24 (GPIO2)
- net GPIO2: now also J1.6 (Pin_6)
- net ID0: now reaches U1.25 (GPIO0)
- net ID0: now also C2.1, D2.1 (K), Q2.1 (C), R5.2, SW2.2
- net GPIO4: now reaches U1.26 (GPIO4)
- net GPIO4: now also J1.5 (Pin_5)
- net GPIO5: now reaches U1.29 (GPIO5)
- net GPIO5: now also J1.7 (Pin_7)
- net EN: now reaches U1.3 (EN)
- net EN: now also C1.1, Q1.1 (C), R3.2, R4.2, SW1.2
- net GPIO18: now reaches U1.30 (GPIO18)
- net GPIO18: now also J1.3 (Pin_3)
- net RXD0: now reaches U1.34 (U0RDX)
- net RXD0: now also R8.2
- net TXD0: now reaches U1.35 (U0TDX)
- net TXD0: now also R9.2
- net GPIO23: now reaches U1.37 (GPIO33)
- net GPIO23: now also J1.4 (Pin_4)
- net HRx: now reaches U1.6 (GPIO34)
- net HRx: now also U3.V2 (V)
- net HRy: now reaches U1.7 (GPIO35)
- net HRy: now also U3.H2 (H)
- new net: Q2.2 (B), R7.2
- new net: Q1.2 (B), R6.2
- new net: D1.2 (A), R2.2
- new net: R8.1, U4.2 (TXD)
- new net: R9.1, U4.3 (RXD)
- new net: D2.2 (A), R1.2
- new net DTR: Q2.3 (E), R6.1, U4.13 (~{DTR})
- new net RTS: Q1.3 (E), R7.1, U4.14 (~{RTS})
- no-connect marks 0 -> 29
Other:
- note added: "BLK"
- note added: "CS"
- note added: "DC"
- note added: "GND"
- note added: "RES"
- note added: "SCL"
- note added: "SDA"
- note added: "VCC"
- moved on the sheet: U1, U2, U3

Commit message: init
Parts:
- added H1, H2, H3, H4: MountingHole, MountingHole:MountingHole_2.2mm_M2_DIN965_Pad, symbol Mechanical:MountingHole

Commit message: init
Parts:
- SW2: value RESET -> BOOT
Connections:
- net +3.3V: now also U2.H2 (H), U2.V2 (V), U3.H2 (H), U3.V2 (V)
- net GND: no longer U2.H1 (H+), U2.V1 (V+), U3.H1 (H+), U3.V1 (V+)
- net HRx: now also U3.V1 (V+); no longer U3.V2 (V)
- net HRy: now also U3.H1 (H+); no longer U3.H2 (H)
- net VRx: now also U2.V1 (V+); no longer U2.V2 (V)
- net VRy: now also U2.H1 (H+); no longer U2.H2 (H)

Commit message: init
Connections:
- net +3.3V: now also J1.7 (Pin_7); no longer J1.2 (Pin_2)
- net GND: now also J1.8 (Pin_8); no longer J1.1 (Pin_1)
- net GPIO15: now also J1.1 (Pin_1); no longer J1.8 (Pin_8)
- net GPIO18: now also J1.6 (Pin_6); no longer J1.3 (Pin_3)
- net GPIO2: now also J1.3 (Pin_3); no longer J1.6 (Pin_6)
- net GPIO23: now also J1.5 (Pin_5); no longer J1.4 (Pin_4)
- net GPIO4: now also J1.4 (Pin_4); no longer J1.5 (Pin_5)
- net GPIO5: now also J1.2 (Pin_2); no longer J1.7 (Pin_7)

Commit message: init
Connections:
- net +3.3V: now also U2.H1 (H+), U2.V1 (V+); no longer U2.H2 (H), U2.V2 (V)
- net VRx: now also U2.V2 (V); no longer U2.V1 (V+)
- net VRy: now also U2.H2 (H); no longer U2.H1 (H+)
Changed lines of the file:
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@@
 	(wire
 		(pts
-			(xy 146.05 44.45) (xy 134.62 44.45)
-		)
-		(stroke
-			(width 0)
-			(type default)
-		)
-	)
-	(wire
-		(pts
 			(xy 100.33 93.98) (xy 102.87 93.98)
 		)
@@
 	(wire
 		(pts
+			(xy 128.27 46.99) (xy 128.27 45.72)
+		)
+		(stroke
+			(width 0)
+			(type default)
+		)
+	)
+	(wire
+		(pts
 			(xy 234.95 68.58) (xy 234.95 72.39)
 		)
@@
 	(wire
 		(pts
+			(xy 133.35 44.45) (xy 146.05 44.45)
+		)
+		(stroke
+			(width 0)
+			(type default)
+		)
+	)
+	(wire
+		(pts
 			(xy 38.1 137.16) (xy 38.1 91.44)
 		)
@@
 	(wire
 		(pts
-			(xy 133.35 46.99) (xy 146.05 46.99)
+			(xy 133.35 88.9) (xy 146.05 88.9)
 		)
 		(stroke
@@
 	(wire
 		(pts
-			(xy 133.35 88.9) (xy 146.05 88.9)
+			(xy 165.1 48.26) (xy 165.1 50.8)
 		)
 		(stroke
@@
 	(wire
 		(pts
-			(xy 165.1 48.26) (xy 165.1 50.8)
+			(xy 196.85 124.46) (xy 204.47 124.46)
 		)
 		(stroke
@@
 	(wire
 		(pts
-			(xy 196.85 124.46) (xy 204.47 124.46)
+			(xy 139.7 49.53) (xy 139.7 53.34)
 		)
 		(stroke
@@
 	(wire
 		(pts
-			(xy 139.7 49.53) (xy 139.7 53.34)
+			(xy 48.26 50.8) (xy 48.26 53.34)
 		)
 		(stroke
@@
 	(wire
 		(pts
-			(xy 48.26 50.8) (xy 48.26 53.34)
+			(xy 209.55 54.61) (xy 209.55 44.45)
 		)
 		(stroke
@@
 	(wire
 		(pts
-			(xy 209.55 54.61) (xy 209.55 44.45)
+			(xy 139.7 39.37) (xy 146.05 39.37)
 		)
 		(stroke
@@
 	(wire
 		(pts
-			(xy 139.7 39.37) (xy 146.05 39.37)
+			(xy 146.05 36.83) (xy 135.89 36.83)
 		)
 		(stroke
@@
 	(wire
 		(pts
-			(xy 133.35 36.83) (xy 146.05 36.83)
+			(xy 240.03 116.84) (xy 243.84 116.84)
 		)
 		(stroke
@@
 	(wire
 		(pts
-			(xy 240.03 116.84) (xy 243.84 116.84)
+			(xy 146.05 46.99) (xy 128.27 46.99)
 		)
 		(stroke
@@
 	(wire
 		(pts
-			(xy 97.79 48.26) (xy 97.79 50.8)
+			(xy 135.89 36.83) (xy 135.89 31.75)
 		)
 		(stroke
@@
 	(wire
 		(pts
-			(xy 236.22 114.3) (xy 240.03 114.3)
+			(xy 97.79 48.26) (xy 97.79 50.8)
 		)
 		(stroke
@@
 	(wire
 		(pts
-			(xy 107.95 107.95) (xy 107.95 109.22)
+			(xy 236.22 114.3) (xy 240.03 114.3)
 		)
 		(stroke
@@
 	(wire
 		(pts
-			(xy 100.33 90.17) (xy 105.41 90.17)
+			(xy 107.95 107.95) (xy 107.95 109.22)
 		)
 		(stroke
@@
 	(wire
 		(pts
-			(xy 31.75 163.83) (xy 31.75 175.26)
+			(xy 100.33 90.17) (xy 105.41 90.17)
 		)
 		(stroke
@@
 	(wire
 		(pts
-			(xy 77.47 100.33) (xy 57.15 100.33)
+			(xy 31.75 163.83) (xy 31.75 175.26)
 		)
 		(stroke
@@
 	(wire
 		(pts
-			(xy 85.09 172.72) (xy 100.33 172.72)
+			(xy 77.47 100.33) (xy 57.15 100.33)
 		)
 		(stroke
@@
 	(wire
 		(pts
-			(xy 138.43 91.44) (xy 146.05 91.44)
+			(xy 85.09 172.72) (xy 100.33 172.72)
 		)
 		(stroke
@@
 	(wire
 		(pts
-			(xy 146.05 34.29) (xy 142.24 34.29)
+			(xy 138.43 91.44) (xy 146.05 91.44)
 		)
 		(stroke
@@
 	(wire
 		(pts
-			(xy 134.62 44.45) (xy 134.62 41.91)
-		)
-		(stroke
-			(width 0)
-			(type default)
-		)
-	)
-	(wire
-		(pts
 			(xy 35.56 50.8) (xy 48.26 50.8)
 		)
@@
 	(wire
 		(pts
-			(xy 142.24 34.29) (xy 142.24 31.75)
-		)
-		(stroke
-			(width 0)
-			(type default)
-		)
-	)
-	(wire
-		(pts
 			(xy 165.1 107.95) (xy 165.1 111.76)
 		)
@@
 	(wire
 		(pts
+			(xy 140.97 34.29) (xy 146.05 34.29)
+		)
+		(stroke
+			(width 0)
+			(type default)
+		)
+	)
+	(wire
+		(pts
 			(xy 240.03 114.3) (xy 240.03 116.84)
 		)
@@
 	)
 	(label "VRx"
-		(at 133.35 36.83 0)
+		(at 140.97 34.29 0)
 		(effects
 			(font
@@
 	)
 	(label "VRy"
-		(at 133.35 46.99 0)
+		(at 133.35 44.45 0)
 		(effects
 			(font
@@
 	(symbol
 		(lib_id "power:+3.3V")
-		(at 134.62 41.91 0)
+		(at 128.27 45.72 0)
 		(unit 1)
 		(exclude_from_sim no)
@@
 		(dnp no)
 		(property "Reference" "#PWR011"
-			(at 134.62 45.72 0)
+			(at 128.27 49.53 0)
 			(effects
 				(font
@@
 		)
 		(property "Value" "+3.3V"
-			(at 130.556 40.64 0)
+			(at 124.206 44.45 0)
 			(effects
 				(font
@@
 		)
 		(property "Footprint" ""
-			(at 134.62 41.91 0)
+			(at 128.27 45.72 0)
 			(effects
 				(font
@@
 		)
 		(property "Datasheet" ""
-			(at 134.62 41.91 0)
+			(at 128.27 45.72 0)
 			(effects
 				(font
@@
 		)
 		(property "Description" "Power symbol creates a global label with name \"+3.3V\""
-			(at 134.62 41.91 0)
+			(at 128.27 45.72 0)
 			(effects
 				(font
@@
 	(symbol
 		(lib_id "power:+3.3V")
-		(at 142.24 31.75 0)
+		(at 135.89 31.75 0)
 		(unit 1)
 		(exclude_from_sim no)
@@
 		(fields_autoplaced yes)
 		(property "Reference" "#PWR016"
-			(at 142.24 35.56 0)
+			(at 135.89 35.56 0)
 			(effects
 				(font
@@
 		)
 		(property "Value" "+3.3V"
-			(at 142.24 26.67 0)
+			(at 135.89 26.67 0)
 			(effects
 				(font
@@
 		)
 		(property "Footprint" ""
-			(at 142.24 31.75 0)
+			(at 135.89 31.75 0)
 			(effects
 				(font
@@
 		)
 		(property "Datasheet" ""
-			(at 142.24 31.75 0)
+			(at 135.89 31.75 0)
 			(effects
 				(font
@@
 		)
 		(property "Description" "Power symbol creates a global label with name \"+3.3V\""
-			(at 142.24 31.75 0)
+			(at 135.89 31.75 0)
 			(effects
 				(font
