File: kicad/esp32-controller.kicad_sch (KiCad schematic)
At the start: 26 parts, among them J1 Conn_01x08_Socket, Q1 BCW66G, Q2 BCW66G, SW1 RESET, SW2 BOOT, U1 ESP32-WROVER-IB, U2 PS4, U3 PS4, U4 CH340C

Commit message: init
Parts:
- removed U2, U3: PS4, PCM_yvolodym:Joystick_PS5, symbol PCM_yvolodym:Joystick_PS5
- added U2, U3: Joystick Analog, PCM_yvolodym:Joystick_Analog, symbol PCM_yvolodym:Joystick_Analog
Connections:
- net +3.3V: now also U2.H1 (H+), U2.V1 (V+), U3.H1 (H+), U3.V1 (V+)
- net GND: now also U2.H3 (H-), U2.S1 (SHIELD), U2.S2 (SHIELD), U2.S3 (SHIELD), U2.S4 (SHIELD), U2.V3 (V-), U3.H3 (H-), U3.S1 (SHIELD), U3.S2 (SHIELD), U3.S3 (SHIELD), U3.S4 (SHIELD), U3.V3 (V-)
- net HRx: now also U3.V2 (V)
- net HRy: now also U3.H2 (H)
- net VRx: now also U2.V2 (V)
- net VRy: now also U2.H2 (H)

Commit message: init
Parts:
- H1, H2, H3, H4: footprint MountingHole:MountingHole_2.2mm_M2_DIN965_Pad -> MountingHole:MountingHole_2.7mm_Pad_Via
Changed lines of the file:
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@@
 			)
 		)
-		(property "Footprint" "MountingHole:MountingHole_2.2mm_M2_DIN965_Pad"
+		(property "Footprint" "MountingHole:MountingHole_2.7mm_Pad_Via"
 			(at 31.75 163.83 0)
 			(effects
@@
 		(dnp no)
 		(property "Reference" "D1"
-			(at 43.942 123.698 0)
+			(at 49.276 122.174 0)
 			(effects
 				(font
@@
 		)
 		(property "Value" "YELLOW"
-			(at 43.942 126.238 0)
+			(at 51.054 124.206 0)
 			(effects
 				(font
@@
 		)
 		(property "Value" "MountingHole"
-			(at 44.45 158.75 0)
+			(at 46.228 158.75 0)
 			(effects
 				(font
@@
 			)
 		)
-		(property "Footprint" "MountingHole:MountingHole_2.2mm_M2_DIN965_Pad"
+		(property "Footprint" "MountingHole:MountingHole_2.7mm_Pad_Via"
 			(at 49.53 163.83 0)
 			(effects
@@
 			)
 		)
-		(property "Footprint" "MountingHole:MountingHole_2.2mm_M2_DIN965_Pad"
+		(property "Footprint" "MountingHole:MountingHole_2.7mm_Pad_Via"
 			(at 40.64 163.83 0)
 			(effects
@@
 			)
 		)
-		(property "Footprint" "MountingHole:MountingHole_2.2mm_M2_DIN965_Pad"
+		(property "Footprint" "MountingHole:MountingHole_2.7mm_Pad_Via"
 			(at 21.59 163.83 0)
 			(effects

Commit message: init
Parts:
- H1, H2, H3, H4: value MountingHole -> MountingHole_Pad; symbol Mechanical:MountingHole -> Mechanical:MountingHole_Pad
Connections:
- net GND: now also H1.1, H2.1, H3.1, H4.1
Changed lines of the file:
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@@
 	)
 	(symbol
-		(lib_id "Mechanical:MountingHole")
-		(at 31.75 163.83 0)
+		(lib_id "Mechanical:MountingHole_Pad")
+		(at 31.75 161.29000000000002 0)
 		(unit 1)
 		(exclude_from_sim yes)
@@
 			)
 		)
-		(property "Value" "MountingHole"
+		(property "Value" "MountingHole_Pad"
 			(at 26.67 158.75 0)
 			(effects
@@
 	)
 	(symbol
-		(lib_id "Mechanical:MountingHole")
-		(at 49.53 163.83 0)
+		(lib_id "Mechanical:MountingHole_Pad")
+		(at 49.53 161.29000000000002 0)
 		(unit 1)
 		(exclude_from_sim yes)
@@
 			)
 		)
-		(property "Value" "MountingHole"
+		(property "Value" "MountingHole_Pad"
 			(at 46.228 158.75 0)
 			(effects
@@
 	)
 	(symbol
-		(lib_id "Mechanical:MountingHole")
-		(at 40.64 163.83 0)
+		(lib_id "Mechanical:MountingHole_Pad")
+		(at 40.64 161.29000000000002 0)
 		(unit 1)
 		(exclude_from_sim yes)
@@
 			)
 		)
-		(property "Value" "MountingHole"
+		(property "Value" "MountingHole_Pad"
 			(at 34.544 167.894 0)
 			(effects
@@
 	)
 	(symbol
-		(lib_id "Mechanical:MountingHole")
-		(at 21.59 163.83 0)
+		(lib_id "Mechanical:MountingHole_Pad")
+		(at 21.59 161.29000000000002 0)
 		(unit 1)
 		(exclude_from_sim yes)
@@
 			)
 		)
-		(property "Value" "MountingHole"
+		(property "Value" "MountingHole_Pad"
 			(at 16.51 167.64 0)
 			(effects
