File: kicad/esp32-controller.kicad_sch (KiCad schematic)
At the start: 26 parts, among them J1 Conn_01x08_Socket, Q1 BCW66G, Q2 BCW66G, SW1 RESET, SW2 BOOT, U1 ESP32-WROVER-IB, U2 Joystick Analog, U3 Joystick Analog, U4 CH340C

Commit message: docu
Parts:
- added C9: 100nF, symbol Device:C
- added R17: 220K, symbol Device:R
- added R18: 100K, symbol Device:R
Connections:
- net GND: now also C9.2, R18.2
- net at U1.4 (SENSOR_VP): now also C9.1, R17.1, R18.1
- new net HVBAT: R17.2
- no-connect marks 29 -> 28
Other:
- sheet supply ports: added HVBAT; removed none

Commit message: docu
Parts:
- renumbered C9 to C1, C1 to C2, C2 to C3, R17 to R1, R8 to R10, R9 to R11, R18 to R2, R1 to R3, R2 to R4, R3 to R5, R4 to R6, R5 to R7, R6 to R8, R7 to R9

Commit message: docu
Parts:
- removed SW1: RESET, Button_Switch_SMD:SW_Push_1P1T_NO_CK_KMR2, symbol Switch:CK_KMS2xxG
- removed SW2: BOOT, Button_Switch_SMD:SW_Push_1P1T_NO_CK_KMR2, symbol Switch:CK_KMS2xxG
- added SW1: RESET, Button_Switch_SMD:SW_SPST_B3U-3000P, symbol Switch:SW_Omron_B3FS
- added SW2: BOOT, Button_Switch_SMD:SW_SPST_B3U-3000P, symbol Switch:SW_Omron_B3FS
- C1: footprint (none) -> Capacitor_SMD:C_1206_3216Metric
- R1, R2: footprint (none) -> Resistor_SMD:R_1206_3216Metric
Connections:
- net EN: now also SW1.2
- net GND: now also SW1.1, SW2.1
- net ID0: now also SW2.2
Changed lines of the file:
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@@
 	)
 	(junction
-		(at 85.09 50.8)
-		(diameter 0)
-		(color 0 0 0 0)
-	)
-	(junction
 		(at 48.26 39.37)
 		(diameter 0)
@@
 	)
 	(junction
-		(at 35.56 50.8)
-		(diameter 0)
-		(color 0 0 0 0)
-	)
-	(junction
 		(at 179.07 52.07)
 		(diameter 0)
@@
 	(wire
 		(pts
-			(xy 85.09 50.8) (xy 97.79 50.8)
+			(xy 77.47 50.8) (xy 97.79 50.8)
 		)
 		(stroke
@@
 	(wire
 		(pts
-			(xy 77.47 50.8) (xy 85.09 50.8)
-		)
-		(stroke
-			(width 0)
-			(type default)
-		)
-	)
-	(wire
-		(pts
 			(xy 179.07 97.79) (xy 179.07 100.33)
 		)
@@
 	(wire
 		(pts
-			(xy 27.94 50.8) (xy 35.56 50.8)
-		)
-		(stroke
-			(width 0)
-			(type default)
-		)
-	)
-	(wire
-		(pts
 			(xy 102.87 92.71) (xy 110.49 92.71)
 		)
@@
 	(wire
 		(pts
-			(xy 85.09 43.18) (xy 85.09 50.8)
-		)
-		(stroke
-			(width 0)
-			(type default)
-		)
-	)
-	(wire
-		(pts
 			(xy 107.95 99.06) (xy 110.49 99.06)
 		)
@@
 	(wire
 		(pts
-			(xy 35.56 50.8) (xy 48.26 50.8)
+			(xy 27.94 50.8) (xy 48.26 50.8)
 		)
 		(stroke
@@
 	(wire
 		(pts
-			(xy 35.56 43.18) (xy 35.56 50.8)
-		)
-		(stroke
-			(width 0)
-			(type default)
-		)
-	)
-	(wire
-		(pts
 			(xy 151.13 45.72) (xy 151.13 48.26)
 		)
@@
 	)
 	(symbol
+		(lib_id "Switch:SW_Omron_B3FS")
+		(at 85.09 39.37 0)
+		(unit 1)
+		(exclude_from_sim no)
+		(in_bom yes)
+		(on_board yes)
+		(dnp no)
+		(fields_autoplaced yes)
+		(property "Reference" "SW2"
+			(at 85.09 31.75 0)
+			(effects
+				(font
+					(size 1.27 1.27)
+				)
+			)
+		)
+		(property "Value" "BOOT"
+			(at 85.09 34.29 0)
+			(effects
+				(font
+					(size 1.27 1.27)
+				)
+			)
+		)
+		(property "Footprint" "Button_Switch_SMD:SW_SPST_B3U-3000P"
+			(at 85.09 34.29 0)
+			(effects
+				(font
+					(size 1.27 1.27)
+				)
+				(hide yes)
+			)
+		)
+		(property "Datasheet" "https://omronfs.omron.com/en_US/ecb/products/pdf/en-b3fs.pdf"
+			(at 85.09 34.29 0)
+			(effects
+				(font
+					(size 1.27 1.27)
+				)
+				(hide yes)
+			)
+		)
+		(property "Description" "Omron B3FS 6x6mm single pole normally-open tactile switch"
+			(at 85.09 39.37 0)
+			(effects
+				(font
+					(size 1.27 1.27)
+				)
+				(hide yes)
+			)
+		)
+		(pin "2"
+		)
+		(pin "1"
+		)
+		(instances
+			(project "esp32-controller"
+				(path "/1b61a099-fa01-45c5-bfa6-c1f023697108"
+					(reference "SW2")
+					(unit 1)
+				)
+			)
+		)
+	)
+	(symbol
 		(lib_id "power:GND")
 		(at 179.07 53.34 0)
@@
 			)
 		)
-		(property "Footprint" ""
+		(property "Footprint" "Resistor_SMD:R_1206_3216Metric"
 			(at 24.638 87.63 90)
 			(effects
@@
 	)
 	(symbol
-		(lib_id "Switch:CK_KMS2xxG")
-		(at 85.09 39.37 0)
-		(unit 1)
-		(exclude_from_sim no)
-		(in_bom yes)
-		(on_board yes)
-		(dnp no)
-		(fields_autoplaced yes)
-		(property "Reference" "SW2"
-			(at 85.09 31.75 0)
-			(effects
-				(font
-					(size 1.27 1.27)
-				)
-			)
-		)
-		(property "Value" "BOOT"
-			(at 85.09 34.29 0)
-			(effects
-				(font
-					(size 1.27 1.27)
-				)
-			)
-		)
-		(property "Footprint" "Button_Switch_SMD:SW_Push_1P1T_NO_CK_KMR2"
-			(at 85.09 34.29 0)
-			(effects
-				(font
-					(size 1.27 1.27)
-				)
-				(hide yes)
-			)
-		)
-		(property "Datasheet" "https://www.ckswitches.com/media/1482/kms.pdf"
-			(at 85.09 34.29 0)
-			(effects
-				(font
-					(size 1.27 1.27)
-				)
-				(hide yes)
-			)
-		)
-		(property "Description" "Microminiature SMT Side Actuated, 4.2 x 2.8 x 1.42mm, without pegs, with shield pin"
-			(at 85.09 39.37 0)
-			(effects
-				(font
-					(size 1.27 1.27)
-				)
-				(hide yes)
-			)
-		)
-		(pin "1"
-		)
-		(pin "SH"
-		)
-		(pin "2"
-		)
-		(instances
-			(project "esp32-controller"
-				(path "/1b61a099-fa01-45c5-bfa6-c1f023697108"
-					(reference "SW2")
-					(unit 1)
-				)
-			)
-		)
-	)
-	(symbol
 		(lib_id "Device:R")
 		(at 218.44 63.5 90)
@@
 	)
 	(symbol
-		(lib_id "Mechanical:MountingHole_Pad")
-		(at 21.59 161.29 0)
+		(lib_id "Switch:SW_Omron_B3FS")
+		(at 35.56 39.37 0)
 		(unit 1)
-		(exclude_from_sim yes)
-		(in_bom no)
+		(exclude_from_sim no)
+		(in_bom yes)
 		(on_board yes)
 		(dnp no)
-		(property "Reference" "H1"
-			(at 24.13 162.5599 0)
+		(fields_autoplaced yes)
+		(property "Reference" "SW1"
+			(at 35.56 31.75 0)
 			(effects
 				(font
 					(size 1.27 1.27)
 				)
-				(justify left)
 			)
 		)
-		(property "Value" "MountingHole_Pad"
-			(at 16.51 167.64 0)
+		(property "Value" "RESET"
+			(at 35.56 34.29 0)
 			(effects
 				(font
 					(size 1.27 1.27)
 				)
-				(justify left)
 			)
 		)
-		(property "Footprint" "MountingHole:MountingHole_2.7mm_Pad_Via"
-			(at 21.59 163.83 0)
+		(property "Footprint" "Button_Switch_SMD:SW_SPST_B3U-3000P"
+			(at 35.56 34.29 0)
 			(effects
 				(font
@@
 			)
 		)
-		(property "Datasheet" "~"
-			(at 21.59 163.83 0)
+		(property "Datasheet" "https://omronfs.omron.com/en_US/ecb/products/pdf/en-b3fs.pdf"
+			(at 35.56 34.29 0)
 			(effects
 				(font
@@
 			)
 		)
-		(property "Description" "Mounting Hole without connection"
-			(at 21.59 163.83 0)
+		(property "Description" "Omron B3FS 6x6mm single pole normally-open tactile switch"
+			(at 35.56 39.37 0)
 			(effects
 				(font
@@
 			)
 		)
+		(pin "2"
+		)
 		(pin "1"
 		)
@@
 			(project "esp32-controller"
 				(path "/1b61a099-fa01-45c5-bfa6-c1f023697108"
-					(reference "H1")
+					(reference "SW1")
 					(unit 1)
 				)
@@
 	)
 	(symbol
-		(lib_id "Switch:CK_KMS2xxG")
-		(at 35.56 39.37 0)
+		(lib_id "Mechanical:MountingHole_Pad")
+		(at 21.59 161.29 0)
 		(unit 1)
-		(exclude_from_sim no)
-		(in_bom yes)
+		(exclude_from_sim yes)
+		(in_bom no)
 		(on_board yes)
 		(dnp no)
-		(fields_autoplaced yes)
-		(property "Reference" "SW1"
-			(at 35.56 31.75 0)
+		(property "Reference" "H1"
+			(at 24.13 162.5599 0)
 			(effects
 				(font
 					(size 1.27 1.27)
 				)
+				(justify left)
 			)
 		)
-		(property "Value" "RESET"
-			(at 35.56 34.29 0)
+		(property "Value" "MountingHole_Pad"
+			(at 16.51 167.64 0)
 			(effects
 				(font
 					(size 1.27 1.27)
 				)
+				(justify left)
 			)
 		)
-		(property "Footprint" "Button_Switch_SMD:SW_Push_1P1T_NO_CK_KMR2"
-			(at 35.56 34.29 0)
+		(property "Footprint" "MountingHole:MountingHole_2.7mm_Pad_Via"
+			(at 21.59 163.83 0)
 			(effects
 				(font
@@
 			)
 		)
-		(property "Datasheet" "https://www.ckswitches.com/media/1482/kms.pdf"
-			(at 35.56 34.29 0)
+		(property "Datasheet" "~"
+			(at 21.59 163.83 0)
 			(effects
 				(font
@@
 			)
 		)
-		(property "Description" "Microminiature SMT Side Actuated, 4.2 x 2.8 x 1.42mm, without pegs, with shield pin"
-			(at 35.56 39.37 0)
+		(property "Description" "Mounting Hole without connection"
+			(at 21.59 163.83 0)
 			(effects
 				(font
@@
 		(pin "1"
 		)
-		(pin "SH"
-		)
-		(pin "2"
-		)
 		(instances
 			(project "esp32-controller"
 				(path "/1b61a099-fa01-45c5-bfa6-c1f023697108"
-					(reference "SW1")
+					(reference "H1")
 					(unit 1)
 				)
@@
 			)
 		)
-		(property "Footprint" ""
+		(property "Footprint" "Resistor_SMD:R_1206_3216Metric"
 			(at 32.258 102.87 90)
 			(effects
@@
 			)
 		)
-		(property "Footprint" ""
+		(property "Footprint" "Capacitor_SMD:C_1206_3216Metric"
 			(at 23.8252 105.41 0)
 			(effects

Commit message: docu
Parts:
- SW1, SW2: footprint Button_Switch_SMD:SW_SPST_B3U-3000P -> Button_Switch_THT:SW_PUSH_1P1T_6x3.5mm_H4.3_APEM_MJTP1243
Changed lines of the file:
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@@
 			)
 		)
-		(property "Footprint" "Button_Switch_SMD:SW_SPST_B3U-3000P"
+		(property "Footprint" "Button_Switch_THT:SW_PUSH_1P1T_6x3.5mm_H4.3_APEM_MJTP1243"
 			(at 85.09 34.29 0)
 			(effects
@@
 			)
 		)
-		(property "Footprint" "Button_Switch_SMD:SW_SPST_B3U-3000P"
+		(property "Footprint" "Button_Switch_THT:SW_PUSH_1P1T_6x3.5mm_H4.3_APEM_MJTP1243"
 			(at 35.56 34.29 0)
 			(effects

Commit message: init
Parts:
- U1: footprint PCM_yvolodym:ESP32-WROVER-B -> PCM_yvolodym:ESP32-WROVER-IB
Changed lines of the file:
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@@
 			)
 		)
-		(property "Footprint" "PCM_yvolodym:ESP32-WROVER-B"
+		(property "Footprint" "PCM_yvolodym:ESP32-WROVER-IB"
 			(at 88.9 86.36 0)
 			(effects
