File: kicad/esp32-controller.kicad_pcb (KiCad board)
At the start: 2 copper layers, 100 x 70 mm, 51 parts, among them J1 Conn_01x08_Socket, J2 Conn_01x02, P1 USB_C_Plug_USB2.0, Q1 BCW66G, Q2 BCW66G, SW1 RESET, SW2 BOOT, U1 ESP32-WROVER-IB, U2 PS4, U3 PS4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

Commit message: init
Parts:
- U10: value ~ -> Switch
- moved D3 40.7 mm to (127.0, 82.0), turned to 90 degrees
- moved R13 21.6 mm to (131.5, 110.5), turned to 180 degrees
- moved R14 19.6 mm to (131.5, 105.0), turned to 0 degrees
- moved SW1 11.1 mm to (169.0, 72.0)
- moved C5 10.3 mm to (186.0, 73.0), turned to 90 degrees
- moved C4 9.30 mm to (193.5, 82.5)
- moved C2 8.99 mm to (193.5, 71.5)
- moved C3 8.92 mm to (193.5, 77.0)
- moved U7 8.65 mm to (194.5, 96.5), turned to -90 degrees
- moved R4 7.26 mm to (171.5, 82.0), turned to 90 degrees
- moved U8 5.72 mm to (186.5, 91.5), turned to 90 degrees
- moved R12 3.83 mm to (138.9, 90.5)
- moved R15 3.83 mm to (145.6, 90.5)
- moved C6 3.80 mm to (186.0, 83.0), turned to 90 degrees
- moved R8 3.70 mm to (178.0, 96.5)
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Connections:
- J1 pad 1: GND -> /GPIO15
- J1 pad 2: +3.3V -> /GPIO5
- J1 pad 3: /GPIO18 -> /GPIO2
- J1 pad 4: /GPIO23 -> /GPIO4
- J1 pad 5: /GPIO4 -> /GPIO23
- J1 pad 6: /GPIO2 -> /GPIO18
- J1 pad 7: /GPIO5 -> +3.3V
- J1 pad 8: /GPIO15 -> GND
Routing:
- net GND: track 0.00 -> 482.5 mm
- net +3.3V: track 0.00 -> 287.3 mm, vias 0 -> 5
- net +5V: track 0.00 -> 162.8 mm, vias 0 -> 3
- net /ID0: track 0.00 -> 115.2 mm, vias 0 -> 5
- net /RTS: track 0.00 -> 90.8 mm, vias 0 -> 3
- net /EN: track 0.00 -> 84.7 mm, vias 0 -> 3
- net Net-(U4-TXD): track 0.00 -> 79.0 mm, vias 0 -> 2
- net /HRx: track 0.00 -> 70.7 mm, vias 0 -> 1
- net /GPIO23: track 0.00 -> 70.3 mm, vias 0 -> 1
- net /DTR: track 0.00 -> 66.5 mm, vias 0 -> 2
- net Net-(U7-S2): track 0.00 -> 61.0 mm, vias 0 -> 1
- net Net-(U4-RXD): track 0.00 -> 58.5 mm, vias 0 -> 2
- net /GPIO5: track 0.00 -> 57.1 mm, vias 0 -> 1
- net Net-(U5-TEMP): track 0.00 -> 56.3 mm, vias 0 -> 3
- net /GPIO2: track 0.00 -> 55.4 mm, vias 0 -> 1
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- added copper zone on F.Cu, net GND
Other:
- board text added: "BLK"
- board text added: "DC"
- board text added: "GND"
- board text added: "RES"
- board text added: "SC"
- board text added: "SCL"
- board text added: "SDA"
- board text added: "VCC"

Commit message: init
Parts:
- moved D1 7.93 mm to (163.0, 83.0)
Connections:
- U2 pad H1: /VRy -> +3.3V
- U2 pad H2: +3.3V -> /VRy
- U2 pad V1: /VRx -> +3.3V
- U2 pad V2: +3.3V -> /VRx
Routing:
- net GND: track 482.5 -> 0.00 mm
- net +3.3V: track 287.3 -> 0.00 mm, vias 5 -> 0
- net +5V: track 162.8 -> 0.00 mm, vias 3 -> 0
- net /ID0: track 115.2 -> 0.00 mm, vias 5 -> 0
- net /RTS: track 90.8 -> 0.00 mm, vias 3 -> 0
- net /EN: track 84.7 -> 0.00 mm, vias 3 -> 0
- net Net-(U4-TXD): track 79.0 -> 0.00 mm, vias 2 -> 0
- net /HRx: track 70.7 -> 0.00 mm, vias 1 -> 0
- net /GPIO23: track 70.3 -> 0.00 mm, vias 1 -> 0
- net /DTR: track 66.5 -> 0.00 mm, vias 2 -> 0
- net Net-(U7-S2): track 61.0 -> 0.00 mm, vias 1 -> 0
- net Net-(U4-RXD): track 58.5 -> 0.00 mm, vias 2 -> 0
- net /GPIO5: track 57.1 -> 0.00 mm, vias 1 -> 0
- net Net-(U5-TEMP): track 56.3 -> 0.00 mm, vias 3 -> 0
- net /GPIO2: track 55.4 -> 0.00 mm, vias 1 -> 0
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
Commit message: init
Parts:
- R12: value 1.2K -> 2K
- R14: value R -> 10K
- U2, U3: value PS4 -> Joystick Analog; footprint PCM_yvolodym:Joystick_PS5 -> PCM_yvolodym:Joystick_Analog
- moved R8 70.9 mm to (114.0, 66.0), turned to 180 degrees
- moved U2 70.7 mm to (115.3, 113.5)
- moved U3 70.0 mm to (184.0, 113.3)
- moved R13 34.5 mm to (104.5, 89.0), turned to -90 degrees
- moved R14 28.2 mm to (144.5, 80.0), turned to 180 degrees
- moved U8 7.62 mm to (193.5, 88.5)
- moved R7 7.57 mm to (185.5, 90.5), turned to 90 degrees
- moved R9 6.82 mm to (133.6, 109.5), turned to -90 degrees
- moved Q1 5.22 mm to (165.0, 108.4), turned to 90 degrees
- moved R6 4.00 mm to (178.0, 90.5), turned to -90 degrees
- moved U10 3.87 mm to (165.5, 123.0)
- moved J2 2.96 mm to (165.9, 98.5)
Connections:
- U3 pad H1: /HRy -> +3.3V
- U3 pad H2: +3.3V -> /HRy
- U3 pad V1: /HRx -> +3.3V
- U3 pad V2: +3.3V -> /HRx

Commit message: init
Parts:
- H1, H2, H3, H4: footprint MountingHole:MountingHole_2.2mm_M2_DIN965_Pad -> MountingHole:MountingHole_2.7mm_Pad_Via
- moved U2 1.20 mm to (116.5, 113.3)
- moved H2 0.50 mm to (104.5, 126.0)
- moved H3 0.50 mm to (195.5, 126.0)

Commit message: init
Parts:
- removed J2: Conn_01x02, Connector_JST:JST_PH_B2B-PH-K_1x02_P2.00mm_Vertical
- added U11: Battary, PCM_yvolodym:NCR18650B, F.Cu at (161.0, 97.5)
- moved U7 7.29 mm to (196.5, 89.5)
- moved U8 2.69 mm to (191.0, 89.5)
Connections:
- U5 pad 1: Net-(U5-TEMP) -> GND
- U5 pad 9: GND -> unconnected-(U5-EPAD-Pad9)_4
- U7 pad 2: unconnected-(U7-D1-Pad2) -> Net-(U7-D1)
- U7 pad 5: unconnected-(U7-D2-Pad5) -> Net-(U7-D1)
Routing:
- net GND: track 0.00 -> 488.9 mm, vias 0 -> 4
- net +3.3V: track 0.00 -> 334.4 mm, vias 0 -> 5
- net +5V: track 0.00 -> 139.4 mm
- net /RTS: track 0.00 -> 117.8 mm, vias 0 -> 5
- net /ID0: track 0.00 -> 112.5 mm, vias 0 -> 4
- net /RXD0: track 0.00 -> 89.8 mm, vias 0 -> 2
- net /EN: track 0.00 -> 82.1 mm, vias 0 -> 4
- net /DTR: track 0.00 -> 81.1 mm, vias 0 -> 2
- net Net-(U7-S2): track 0.00 -> 67.8 mm, vias 0 -> 3
- net Net-(U10-Pad2): track 0.00 -> 64.2 mm, vias 0 -> 1
- net /GPIO5: track 0.00 -> 64.2 mm, vias 0 -> 2
- net /GPIO18: track 0.00 -> 58.7 mm, vias 0 -> 1
- net /GPIO23: track 0.00 -> 57.1 mm, vias 0 -> 1
- net /VRx: track 0.00 -> 56.4 mm, vias 0 -> 2
- net /VRy: track 0.00 -> 53.5 mm, vias 0 -> 2
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- removed copper zone on F.Cu, net GND

Commit message: init
Parts:
- D5: value LED -> BLAU
- U11: moved to B.Cu
- moved R7 17.9 mm to (168.5, 96.0)
- moved U8 11.5 mm to (179.5, 90.0), turned to 180 degrees
- moved C6 10.0 mm to (196.0, 84.0), turned to 180 degrees
- moved C4 7.65 mm to (186.0, 84.0)
- moved U7 7.02 mm to (189.5, 90.0), turned to 0 degrees
- moved R6 6.52 mm to (174.5, 96.0)
- moved C3 1.80 mm to (192.0, 78.0)
- turned U11 to 180 degrees
Routing:
- net /RTS: track 117.8 -> 81.2 mm, vias 5 -> 2
- net +3.3V: track 334.4 -> 315.0 mm, vias 5 -> 4
- net Net-(D4-K): track 33.4 -> 15.3 mm
- net /RXD0: track 89.8 -> 71.7 mm
- net Net-(P1-D+): track 17.4 -> 31.2 mm, vias 0 -> 2
- net /EN: track 82.1 -> 94.7 mm, vias 4 -> 3
- net Net-(Q2-B): track 16.9 -> 4.74 mm
- net Net-(U7-G2): track 6.55 -> 18.4 mm
- net Net-(P1-D-): track 28.2 -> 16.9 mm, vias 2 -> 0
- net /DTR: track 81.1 -> 70.7 mm
- net Net-(U10-Pad2): track 64.2 -> 54.1 mm
- net Net-(Q1-B): track 24.9 -> 15.5 mm, vias 2 -> 0
- net GND: track 488.9 -> 498.1 mm, vias 4 -> 5
- net /ID0: track 112.5 -> 121.6 mm, vias 4 -> 3
- net +5V: track 139.4 -> 148.0 mm, vias 0 -> 3
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- added copper zone on F.Cu, net GND
