File: kicad/esp32-controller.kicad_pcb (KiCad board)
At the start: 2 copper layers, 100 x 70 mm, 51 parts, among them J1 Conn_01x08_Socket, P1 USB_C_Plug_USB2.0, Q1 BCW66G, Q2 BCW66G, SW1 RESET, SW2 BOOT, U1 ESP32-WROVER-IB, U10 Switch, U11 Battary, U2 Joystick Analog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

Commit message: init
Parts:
- removed R14: 10K, Resistor_SMD:R_1206_3216Metric
- removed R15: R, Resistor_SMD:R_1206_3216Metric
- moved U10 61.0 mm to (187.0, 66.0), turned to 90 degrees
- moved R10 56.3 mm to (181.0, 81.5)
- moved Q1 49.5 mm to (126.0, 78.0), turned to 0 degrees
- moved R6 46.7 mm to (132.5, 75.5)
- moved C6 44.1 mm to (152.0, 81.0), turned to -90 degrees
- moved Q2 42.5 mm to (127.5, 87.0), turned to 90 degrees
- moved U7 42.4 mm to (150.0, 74.5), turned to 180 degrees
- moved R7 38.1 mm to (133.5, 81.0), turned to -90 degrees
- moved R17 37.6 mm to (194.5, 103.0)
- moved R12 35.6 mm to (174.0, 84.5), turned to -90 degrees
- moved U8 35.4 mm to (145.5, 80.0), turned to 0 degrees
- moved C2 34.5 mm to (161.5, 84.5), turned to -90 degrees
- moved R8 30.0 mm to (140.0, 81.0), turned to -90 degrees
- moved U5 29.7 mm to (162.3, 92.7), turned to 180 degrees
- moved D3 26.6 mm to (104.0, 95.3), turned to -90 degrees
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Routing:
- net GND: track 498.1 -> 0.00 mm, vias 5 -> 0
- net +3.3V: track 315.0 -> 0.00 mm, vias 4 -> 0
- net +5V: track 148.0 -> 0.00 mm, vias 3 -> 0
- net /ID0: track 121.6 -> 0.00 mm, vias 3 -> 0
- net /EN: track 94.7 -> 0.00 mm, vias 3 -> 0
- net /RTS: track 81.2 -> 0.00 mm, vias 2 -> 0
- net /RXD0: track 71.7 -> 0.00 mm, vias 2 -> 0
- net /DTR: track 70.7 -> 0.00 mm, vias 2 -> 0
- net Net-(U7-S2): track 63.1 -> 0.00 mm, vias 1 -> 0
- net /GPIO5: track 60.1 -> 0.00 mm, vias 1 -> 0
- net /GPIO23: track 57.9 -> 0.00 mm, vias 1 -> 0
- net /GPIO15: track 55.8 -> 0.00 mm, vias 1 -> 0
- net /VRy: track 55.5 -> 0.00 mm, vias 2 -> 0
- net Net-(U10-Pad2): track 54.1 -> 0.00 mm, vias 1 -> 0
- net /VRx: track 53.1 -> 0.00 mm, vias 2 -> 0
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
Commit message: init
Parts:
- removed D5: BLAU, Diode_SMD:D_0603_1608Metric
- removed R16: 1K, Resistor_SMD:R_1206_3216Metric
- removed R17: 100, Resistor_SMD:R_1206_3216Metric
- added R14: 100, Resistor_SMD:R_1206_3216Metric, F.Cu at (123.5, 94.5)
- D3: value GREEN -> RED
- D4: value RED -> BLAU
- R11: value 1K -> 2K
- R13: value 2K -> 1K
- moved D4 64.6 mm to (175.8, 82.5), turned to 0 degrees
- moved R10 38.7 mm to (144.5, 94.5), turned to 180 degrees
- moved D3 37.7 mm to (141.0, 88.0), turned to 90 degrees
- moved R12 6.91 mm to (180.0, 88.0), turned to 180 degrees
- moved U11 0.50 mm to (158.5, 82.0)
Connections:
- D4 pad 1: Net-(D4-K) -> GND
- D4 pad 2: +5V -> Net-(D4-A)
- R10 pad 1: Net-(U5-~{STDBY}) -> Net-(U5-~{CHRG})
- R11 pad 1: Net-(U5-~{CHRG}) -> GND
- R11 pad 2: Net-(D4-K) -> Net-(U5-PROG)
- R12 pad 1: GND -> +5V
- R12 pad 2: Net-(U5-PROG) -> Net-(D4-A)
- R13 pad 1: +5V -> GND
- R13 pad 2: Net-(D5-A) -> Net-(U8-CS)
- U5 pad 6: Net-(U5-~{STDBY}) -> GND
Routing:
- net GND: track 0.00 -> 506.3 mm, vias 0 -> 8
- net +3.3V: track 0.00 -> 274.7 mm, vias 0 -> 3
- net /EN: track 0.00 -> 161.4 mm, vias 0 -> 5
- net /ID0: track 0.00 -> 141.7 mm, vias 0 -> 4
- net +5V: track 0.00 -> 106.3 mm, vias 0 -> 3
- net /GPIO5: track 0.00 -> 67.0 mm, vias 0 -> 1
- net /GPIO23: track 0.00 -> 63.8 mm, vias 0 -> 1
- net /GPIO15: track 0.00 -> 58.2 mm, vias 0 -> 1
- net Net-(U7-S2): track 0.00 -> 57.1 mm, vias 0 -> 2
- net Net-(U8-CS): track 0.00 -> 55.2 mm, vias 0 -> 2
- net /VRx: track 0.00 -> 54.0 mm, vias 0 -> 2
- net /GPIO4: track 0.00 -> 51.7 mm, vias 0 -> 1
- net /VRy: track 0.00 -> 50.5 mm, vias 0 -> 2
- net /GPIO18: track 0.00 -> 50.1 mm, vias 0 -> 2
- net /GPIO2: track 0.00 -> 48.2 mm, vias 0 -> 1
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
Commit message: init
Other:
- board text added: "Version 3"
Changed lines of the file:
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@@
+		)
+	)
+	(gr_text "Version 3"
+		(at 198 116 90)
+		(layer "F.SilkS")
+		(effects
+			(font
+				(size 1.5 1.5)
+				(thickness 0.3)
+				(bold yes)
+			)
+			(justify left bottom)
 		)
 	)

Commit message: init
Parts:
- removed SW1: RESET, Button_Switch_SMD:SW_Push_1P1T_NO_CK_KMR2
- removed SW2: BOOT, Button_Switch_SMD:SW_Push_1P1T_NO_CK_KMR2
- added BOOT: BOOT, Button_Switch_SMD:SW_Push_1P1T_NO_CK_KMR2, F.Cu at (171.0, 65.0)
- added D5: SS14, Diode_SMD:D_SMA, F.Cu at (174.5, 91.5)
- added D6: SS14, Diode_SMD:D_SMA, F.Cu at (172.0, 78.0)
- added Q3: Si2319CDS, Package_TO_SOT_SMD:SOT-23, F.Cu at (151.9, 92.0)
- added R15: 1K, Resistor_SMD:R_1206_3216Metric, F.Cu at (162.5, 73.0)
- added R16: 100, Resistor_SMD:R_1206_3216Metric, F.Cu at (167.0, 73.0)
- added RESET: RESET, Button_Switch_SMD:SW_Push_1P1T_NO_CK_KMR2, F.Cu at (163.0, 65.0)
- added U12: LTC4412, Package_TO_SOT_SMD:TSOT-23-6, F.Cu at (142.5, 92.0)
- H1, H2, H3, H4: value MountingHole -> MountingHole_Pad
- R11, R12: value 2K -> 5.1k
- R13: value 1K -> 2K
- R14: value 100 -> 2K
- U10: value Switch -> Battery; footprint PCM_yvolodym:Switch -> PCM_yvolodym:NCR18650B; moved to B.Cu
- U11: value Battary -> AP2112K-3.3; footprint PCM_yvolodym:NCR18650B -> Package_TO_SOT_SMD:SOT-23-5; moved to F.Cu
- U9: value AMS1117-3.3 -> Switch; footprint Package_TO_SOT_SMD:SOT-223-3_TabPin2 -> PCM_yvolodym:Switch
- moved R13 52.0 mm to (153.0, 73.0)
- moved C8 47.5 mm to (193.5, 99.5), turned to 0 degrees
- moved D3 46.7 mm to (186.3, 76.4), turned to 0 degrees
- moved R14 40.7 mm to (158.0, 73.0), turned to 90 degrees
- moved R5 36.7 mm to (159.5, 84.5), turned to -90 degrees
- moved R7 36.7 mm to (170.0, 84.5)
- moved R4 36.3 mm to (154.5, 84.5)
- moved R3 35.8 mm to (149.5, 84.5)
- moved R12 35.3 mm to (148.0, 73.0), turned to 90 degrees
- moved Q2 34.8 mm to (161.9, 92.0), turned to 0 degrees
- moved U10 33.6 mm to (159.0, 84.5), turned to 180 degrees
- moved C6 33.4 mm to (183.5, 70.0), turned to 0 degrees
- moved R6 33.2 mm to (164.5, 84.5), turned to 90 degrees
- moved U5 32.2 mm to (130.3, 89.2), turned to 0 degrees
- moved C2 31.5 mm to (192.0, 92.5), turned to 0 degrees
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Connections:
- C4 pad 1: +3.3V -> /supply/VBAT
- H1 pad 1: (no net) -> GND
- H2 pad 1: (no net) -> GND
- H3 pad 1: (no net) -> GND
- H4 pad 1: (no net) -> GND
- P1 pad A5: unconnected-(P1-CC-PadA5) -> Net-(P1-CC)
- P1 pad B5: unconnected-(P1-VCONN-PadB5) -> Net-(P1-VCONN)
- R11 pad 1: GND -> Net-(P1-CC)
- R11 pad 2: Net-(U5-PROG) -> GND
- R12 pad 1: +5V -> Net-(P1-VCONN)
- R12 pad 2: Net-(D4-A) -> GND
- R13 pad 2: Net-(U8-CS) -> Net-(U5-PROG)
- R14 pad 1: +3.3V -> +5V
- R14 pad 2: Net-(U8-VCC) -> Net-(D4-A)
- U10 pad 1: unconnected-(U10-Pad1) -> /supply/VBAT
- U11 pad 1: +3.3V -> /supply/VPWR
- U11 pad 2: Net-(U10-Pad2) -> GND
- U5 pad 1: GND -> +5V
- U5 pad 5: +3.3V -> /supply/VBAT
- U5 pad 6: GND -> unconnected-(U5-~{STDBY}-Pad6)
- U5 pad 9: unconnected-(U5-EPAD-Pad9)_6 -> GND
- U9 pad 1: GND -> unconnected-(U9-Pad1)
- U9 pad 2: +3.3V -> Net-(U10-Pad2)
- U9 pad 3: +5V -> Net-(U7-S2)
Routing:
- net GND: track 506.3 -> 0.00 mm, vias 8 -> 0
- net +3.3V: track 274.7 -> 0.00 mm, vias 3 -> 0
- net /EN: track 161.4 -> 0.00 mm, vias 5 -> 0
- net /ID0: track 141.7 -> 0.00 mm, vias 4 -> 0
- net +5V: track 106.3 -> 0.00 mm, vias 3 -> 0
- net /GPIO5: track 67.0 -> 0.00 mm, vias 1 -> 0
- net /GPIO23: track 63.8 -> 0.00 mm, vias 1 -> 0
- net /GPIO15: track 58.2 -> 0.00 mm, vias 1 -> 0
- net Net-(U7-S2): track 57.1 -> 0.00 mm, vias 2 -> 0
- net Net-(U8-CS): track 55.2 -> 0.00 mm, vias 2 -> 0
- net /VRx: track 54.0 -> 0.00 mm, vias 2 -> 0
- net /GPIO4: track 51.7 -> 0.00 mm, vias 1 -> 0
- net /VRy: track 50.5 -> 0.00 mm, vias 2 -> 0
- net /GPIO18: track 50.1 -> 0.00 mm, vias 2 -> 0
- net /GPIO2: track 48.2 -> 0.00 mm, vias 1 -> 0
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- removed copper zone on F.Cu, net GND
Other:
- board text added: "Version 4"
- board text removed: "Version 3"

Commit message: init
Parts:
- moved C4 5.72 mm to (188.0, 85.0), turned to 0 degrees
- moved U9 5.59 mm to (185.0, 64.0), turned to 90 degrees
- moved U4 5.06 mm to (125.5, 69.5)
- moved U10 1.12 mm to (159.5, 83.5)
- turned U12 to 180 degrees
Routing:
- net GND: track 0.00 -> 576.9 mm, vias 0 -> 2
- net +3.3V: track 0.00 -> 228.7 mm
- net +5V: track 0.00 -> 166.5 mm, vias 0 -> 3
- net /ID0: track 0.00 -> 127.4 mm, vias 0 -> 5
- net /EN: track 0.00 -> 104.2 mm, vias 0 -> 4
- net /supply/VBAT: track 0.00 -> 88.8 mm
- net /GPIO23: track 0.00 -> 63.5 mm, vias 0 -> 1
- net Net-(D3-K): track 0.00 -> 62.9 mm, vias 0 -> 2
- net /DTR: track 0.00 -> 60.6 mm, vias 0 -> 2
- net /VRx: track 0.00 -> 56.2 mm
- net /GPIO5: track 0.00 -> 53.2 mm, vias 0 -> 1
- net /RTS: track 0.00 -> 48.9 mm, vias 0 -> 2
- net Net-(U4-TXD): track 0.00 -> 48.3 mm, vias 0 -> 2
- net /GPIO15: track 0.00 -> 47.7 mm, vias 0 -> 1
- net /GPIO4: track 0.00 -> 44.4 mm
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- added copper zone on F.Cu, net GND

Commit message: docu
Parts:
- removed BOOT: BOOT, Button_Switch_SMD:SW_Push_1P1T_NO_CK_KMR2
- removed D6: SS14, Diode_SMD:D_SMA
- removed RESET: RESET, Button_Switch_SMD:SW_Push_1P1T_NO_CK_KMR2
- added C9: 100nF, Capacitor_SMD:C_1206_3216Metric, F.Cu at (175.7, 84.5)
- added R17: 1K, Resistor_SMD:R_1206_3216Metric, F.Cu at (181.0, 84.5)
- added R18: 100, Resistor_SMD:R_1206_3216Metric, F.Cu at (192.0, 84.0)
- added SW1: RESET, Button_Switch_SMD:SW_Push_1P1T_NO_CK_KMR2, F.Cu at (155.7, 65.0)
- added SW2: BOOT, Button_Switch_SMD:SW_Push_1P1T_NO_CK_KMR2, F.Cu at (162.7, 65.0)
- C3, C7: value 10µF -> 100nF
- C6: value 100pF -> 10µF
- C8: value 100nF -> 10µF
- R1: value 2K -> 220K
- R10: value 1K -> 470
- R11: value 5.1k -> 470
- R12: value 5.1k -> 1K
- R13, R14: value 2K -> 5.1k
- R15: value 1K -> 2K
- R16: value 100 -> 2K
- R2: value 2K -> 100K
- R3, R4: value 10K -> 2K
- R8, R9: value 470 -> 10K
- moved D2 43.8 mm to (106.4, 97.0), turned to 90 degrees
- moved D4 35.3 mm to (186.3, 82.5)
- moved U7 7.27 mm to (172.4, 78.0)
- moved C4 6.02 mm to (184.0, 89.5)
- moved C3 5.61 mm to (180.0, 77.5)
- moved C2 2.53 mm to (192.0, 90.0), turned to 90 degrees
- moved R6 0.64 mm to (165.1, 84.5)
- moved R14 0.50 mm to (157.5, 73.0)
- moved R7 0.43 mm to (170.4, 84.5)
- moved R5 0.36 mm to (159.9, 84.5)
- moved R11 0.25 mm to (143.2, 73.0)
- moved R13 0.25 mm to (152.8, 73.0)
- moved R15 0.25 mm to (162.2, 73.0)
- moved R3 0.21 mm to (149.3, 84.5)
- moved R4 0.07 mm to (154.6, 84.5)
Connections:
- C1 pad 1: /EN -> Net-(U1-SENSOR_VP)
- C2 pad 1: /ID0 -> /EN
- C3 pad 1: +5V -> /ID0
- C4 pad 1: /supply/VBAT -> +5V
- C5 pad 1: +5V -> /HVBAT
- C6 pad 1: Net-(U7-S2) -> +5V
- C6 pad 2: Net-(U8-VCC) -> GND
- C7 pad 1: +3.3V -> Net-(U7-S2)
- C7 pad 2: GND -> Net-(U8-VCC)
- C8 pad 1: GND -> +3.3V
- C8 pad 2: +5V -> GND
- Q3 pad 2: Net-(D6-K) -> /supply/VPWR
- Q3 pad 3: /supply/VPWR -> /HVBAT
- R1 pad 1: +3.3V -> Net-(U1-SENSOR_VP)
- R1 pad 2: Net-(D2-A) -> /HVBAT
- R10 pad 1: Net-(U5-~{CHRG}) -> Net-(U4-TXD)
- R10 pad 2: Net-(D3-K) -> /RXD0
- R11 pad 1: Net-(P1-CC) -> Net-(U4-RXD)
- R11 pad 2: GND -> /TXD0
- R12 pad 1: Net-(P1-VCONN) -> Net-(U5-~{CHRG})
- R12 pad 2: GND -> Net-(D3-K)
- R13 pad 1: GND -> Net-(P1-CC)
- R13 pad 2: Net-(U5-PROG) -> GND
- R14 pad 1: +5V -> Net-(P1-VCONN)
- R14 pad 2: Net-(D4-A) -> GND
- R15 pad 2: Net-(U8-CS) -> Net-(U5-PROG)
- R16 pad 1: /supply/VBAT -> +5V
- R16 pad 2: Net-(U8-VCC) -> Net-(D4-A)
- R2 pad 1: +3.3V -> Net-(U1-SENSOR_VP)
- R2 pad 2: Net-(D1-A) -> GND
- R3 pad 2: /EN -> Net-(D2-A)
- R4 pad 2: /EN -> Net-(D1-A)
- R5 pad 2: /ID0 -> /EN
- R6 pad 1: /DTR -> +3.3V
- R6 pad 2: Net-(Q1-B) -> /EN
- R7 pad 1: /RTS -> +3.3V
- R7 pad 2: Net-(Q2-B) -> /ID0
- R8 pad 1: Net-(U4-TXD) -> /DTR
- R8 pad 2: /RXD0 -> Net-(Q1-B)
- R9 pad 1: Net-(U4-RXD) -> /RTS
- R9 pad 2: /TXD0 -> Net-(Q2-B)
- U1 pad 4: unconnected-(U1-SENSOR_VP-Pad4) -> Net-(U1-SENSOR_VP)
- U10 pad 1: /supply/VBAT -> /HVBAT
- U12 pad 1: /supply/VBAT -> /HVBAT
- U5 pad 5: /supply/VBAT -> /HVBAT
Routing:
- net GND: track 576.9 -> 0.70 mm, vias 2 -> 0
- net /HVBAT: track 0.00 -> 109.2 mm, vias 0 -> 3
- net Net-(U1-SENSOR_VP): track 0.00 -> 98.2 mm, vias 0 -> 4
- net /supply/VBAT: track 88.8 -> 0.00 mm
- net Net-(Q1-B): track 11.8 -> 56.8 mm, vias 0 -> 2
- net Net-(D2-A): track 7.61 -> 49.1 mm
- net /DTR: track 60.6 -> 100.1 mm, vias 2 -> 3
- net /RXD0: track 14.5 -> 47.7 mm, vias 0 -> 2
- net Net-(D6-K): track 29.6 -> 0.00 mm, vias 2 -> 0
- net Net-(U7-S2): track 29.7 -> 59.2 mm, vias 1 -> 2
- net Net-(U4-TXD): track 48.3 -> 18.8 mm
- net /TXD0: track 23.3 -> 51.4 mm
- net Net-(D1-A): track 5.93 -> 33.0 mm, vias 0 -> 2
- net +5V: track 166.5 -> 142.8 mm, vias 3 -> 5
- net Net-(P1-D+): track 42.7 -> 21.1 mm, vias 0 -> 2
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Other:
- board text added: "Version 5"
- board text removed: "Version 4"

Commit message: docu
Parts:
- R16: value 2K -> 470
- moved R18 6.96 mm to (189.5, 90.5)
- moved C2 2.55 mm to (194.5, 90.5), turned to -90 degrees
- moved D3 2.21 mm to (188.2, 77.5)
- moved D4 2.21 mm to (188.2, 83.6)
- moved C5 1.41 mm to (194.5, 77.0)
- moved C4 0.69 mm to (184.5, 90.0), turned to 90 degrees
Connections:
- net /supply/Q1_GATE renamed Net-(Q3-G)
- net /supply/VPWR renamed Net-(D5-K)
- R16 pad 1: +5V -> +3.3V
Routing:
- net +3.3V: track 246.0 -> 0.00 mm
- net +5V: track 142.8 -> 0.00 mm, vias 5 -> 0
- net /ID0: track 128.0 -> 0.00 mm, vias 4 -> 0
- net /EN: track 112.5 -> 0.00 mm, vias 4 -> 0
- net /HVBAT: track 109.2 -> 0.00 mm, vias 3 -> 0
- net /DTR: track 100.1 -> 0.00 mm, vias 3 -> 0
- net Net-(U1-SENSOR_VP): track 98.2 -> 0.00 mm, vias 4 -> 0
- net /RTS: track 69.5 -> 0.00 mm, vias 2 -> 0
- net Net-(U7-S2): track 59.2 -> 0.00 mm, vias 2 -> 0
- net Net-(Q1-B): track 56.8 -> 0.00 mm, vias 2 -> 0
- net /VRx: track 55.5 -> 0.00 mm
- net /GPIO23: track 53.6 -> 0.00 mm, vias 1 -> 0
- net /TXD0: track 51.4 -> 0.00 mm, vias 2 -> 0
- net Net-(D3-K): track 50.1 -> 0.00 mm, vias 2 -> 0
- net Net-(U5-PROG): track 49.8 -> 0.00 mm, vias 2 -> 0
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
Commit message: init
Parts:
- D3: value RED -> LED_RED; footprint Diode_SMD:D_0603_1608Metric -> LED_THT:LED_D2.0mm_W4.8mm_H2.5mm_FlatTop
- D4: value BLAU -> LED_GREEN; footprint Diode_SMD:D_0603_1608Metric -> LED_THT:LED_D2.0mm_W4.8mm_H2.5mm_FlatTop
- moved D3 2.04 mm to (186.2, 77.0)
- moved D4 1.98 mm to (186.2, 83.6)
- moved C6 1.50 mm to (183.5, 71.5), turned to 180 degrees
- turned C5 to 90 degrees
