File: kicad/esp32-controller.kicad_pcb (KiCad board)
At the start: 2 copper layers, 100 x 70 mm, 55 parts, among them J1 Conn_01x08_Socket, P1 USB_C_Plug_USB2.0, Q1 BCW66G, Q2 BCW66G, Q3 Si2319CDS, SW1 RESET, SW2 BOOT, U1 ESP32-WROVER-IB, U10 Battery, U11 AP2112K-3.3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

Commit message: docu
Parts:
- D4: value LED_GREEN -> SS14; footprint LED_THT:LED_D2.0mm_W4.8mm_H2.5mm_FlatTop -> Diode_SMD:D_SMA
- D5: value SS14 -> LED_GREEN; footprint Diode_SMD:D_SMA -> LED_THT:LED_D2.0mm_W4.8mm_H2.5mm_FlatTop
- R16: value 470 -> 1K
- R17: value 1K -> 100
- R18: value 100 -> 470
- SW1, SW2: footprint Button_Switch_SMD:SW_Push_1P1T_NO_CK_KMR2 -> Button_Switch_SMD:SW_SPST_B3U-3000P
- U10: value Battery -> Switch; footprint PCM_yvolodym:NCR18650B -> PCM_yvolodym:Switch
- U11: value AP2112K-3.3 -> Battery; footprint Package_TO_SOT_SMD:SOT-23-5 -> PCM_yvolodym:NCR18650B
- U12: value LTC4412 -> AP2112K-3.3; footprint Package_TO_SOT_SMD:TSOT-23-6 -> Package_TO_SOT_SMD:SOT-23-5
- U9: value Switch -> LTC4412; footprint PCM_yvolodym:Switch -> Package_TO_SOT_SMD:TSOT-23-6
- moved U10 21.3 mm to (168.0, 64.0), turned to 90 degrees
- moved SW2 8.92 mm to (153.8, 64.5), turned to 0 degrees
- moved SW1 4.63 mm to (160.3, 64.5), turned to 0 degrees
Connections:
- D4 pad 1: GND -> Net-(D4-K)
- D4 pad 2: Net-(D4-A) -> +5V
- D5 pad 1: Net-(D5-K) -> GND
- D5 pad 2: +5V -> Net-(D5-A)
- Q3 pad 2: Net-(D5-K) -> Net-(D4-K)
- R16 pad 1: +3.3V -> GND
- R16 pad 2: Net-(D4-A) -> Net-(U8-CS)
- R17 pad 1: GND -> /HVBAT
- R17 pad 2: Net-(U8-CS) -> Net-(U8-VCC)
- R18 pad 1: /HVBAT -> +3.3V
- R18 pad 2: Net-(U8-VCC) -> Net-(D5-A)
- U10 pad 1: /HVBAT -> unconnected-(U10-Pad1)
- U11 pad 1: Net-(D5-K) -> /HVBAT
- U11 pad 2: GND -> Net-(U10-Pad2)
- U12 pad 1: /HVBAT -> Net-(D4-K)
- U12 pad 3: GND -> Net-(D4-K)
- U12 pad 5: Net-(Q3-G) -> +3.3V
- U9 pad 1: unconnected-(U9-Pad1) -> /HVBAT
- U9 pad 2: Net-(U10-Pad2) -> GND
- U9 pad 3: Net-(U7-S2) -> GND

Commit message: docu
Parts:
- SW1, SW2: footprint Button_Switch_SMD:SW_SPST_B3U-3000P -> Button_Switch_THT:SW_PUSH_1P1T_6x3.5mm_H4.3_APEM_MJTP1243
- U10: footprint PCM_yvolodym:Switch -> Button_Switch_SMD:SW_SPDT_PCM12; moved to F.Cu
- moved U10 7.50 mm to (175.5, 63.8), turned to 180 degrees
- moved SW1 2.26 mm to (162.5, 64.0)
- moved SW2 1.87 mm to (152.0, 64.0)

Commit message: init
Parts:
- moved D4 71.8 mm to (115.5, 96.0), turned to 180 degrees
- moved U11 16.6 mm to (160.2, 83.0)
- moved D5 14.4 mm to (186.5, 83.5)
- moved C9 4.17 mm to (171.6, 85.0)
- moved R1 4.17 mm to (139.9, 85.0)
- moved R17 4.17 mm to (176.9, 85.0)
- moved R3 4.17 mm to (145.1, 85.0)
- moved R4 4.17 mm to (150.4, 85.0)
- moved R5 4.17 mm to (155.7, 85.0)
- moved R6 4.17 mm to (161.0, 85.0)
- moved R7 4.17 mm to (166.3, 85.0)
- moved D3 0.23 mm to (186.5, 77.0)

Commit message: init
Parts:
- U1: footprint PCM_yvolodym:ESP32-WROVER-B -> PCM_yvolodym:ESP32-WROVER-IB
- U11: moved to B.Cu
- moved C7 9.16 mm to (173.5, 91.0)
- moved C2 7.50 mm to (187.0, 90.5)
- moved C4 2.54 mm to (182.0, 90.5)
- moved R18 2.50 mm to (192.0, 90.5)
- moved U8 0.71 mm to (175.1, 71.5)
- turned U11 to 180 degrees
Routing:
- net +3.3V: track 0.00 -> 269.1 mm
- net +5V: track 0.00 -> 152.8 mm, vias 0 -> 2
- net /HVBAT: track 0.00 -> 131.2 mm, vias 0 -> 4
- net /ID0: track 0.00 -> 129.3 mm, vias 0 -> 4
- net /EN: track 0.00 -> 119.3 mm, vias 0 -> 3
- net Net-(U1-SENSOR_VP): track 0.00 -> 118.7 mm, vias 0 -> 4
- net Net-(D4-K): track 0.00 -> 94.2 mm, vias 0 -> 2
- net /DTR: track 0.00 -> 74.8 mm, vias 0 -> 3
- net /RTS: track 0.00 -> 64.8 mm, vias 0 -> 3
- net Net-(Q3-G): track 0.00 -> 61.1 mm, vias 0 -> 2
- net /GPIO5: track 0.00 -> 60.5 mm, vias 0 -> 1
- net Net-(U5-PROG): track 0.00 -> 60.1 mm, vias 0 -> 2
- net /VRx: track 0.00 -> 55.4 mm
- net Net-(D3-K): track 0.00 -> 55.0 mm, vias 0 -> 1
- net /TXD0: track 0.00 -> 53.1 mm, vias 0 -> 2
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
Commit message: init
Routing:
- net +3.3V: track 269.1 -> 0.00 mm
- net +5V: track 152.8 -> 0.00 mm, vias 2 -> 0
- net /HVBAT: track 131.2 -> 0.00 mm, vias 4 -> 0
- net /ID0: track 129.3 -> 0.00 mm, vias 4 -> 0
- net /EN: track 119.3 -> 0.00 mm, vias 3 -> 0
- net Net-(U1-SENSOR_VP): track 118.7 -> 0.00 mm, vias 4 -> 0
- net Net-(D4-K): track 94.2 -> 0.00 mm, vias 2 -> 0
- net /DTR: track 74.8 -> 0.00 mm, vias 3 -> 0
- net /RTS: track 64.8 -> 0.00 mm, vias 3 -> 0
- net Net-(Q3-G): track 61.1 -> 0.00 mm, vias 2 -> 0
- net /GPIO5: track 60.5 -> 0.00 mm, vias 1 -> 0
- net Net-(U5-PROG): track 60.1 -> 0.00 mm, vias 2 -> 0
- net /VRx: track 55.4 -> 0.00 mm
- net Net-(D3-K): track 55.0 -> 0.00 mm, vias 1 -> 0
- net /TXD0: track 53.1 -> 0.00 mm, vias 2 -> 0
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
Commit message: init
Parts:
- moved Q1 32.3 mm to (128.5, 97.5)
- moved R10 3.91 mm to (136.8, 76.5)
- moved R11 3.91 mm to (141.5, 76.5)
- moved R12 3.91 mm to (146.2, 76.5)
- moved R13 3.91 mm to (151.0, 76.5)
- moved R14 3.91 mm to (155.8, 76.5)
- moved R15 3.91 mm to (160.5, 76.5)
- moved R16 3.91 mm to (165.2, 76.5)
- moved U6 3.31 mm to (128.9, 78.5)
- moved U4 2.97 mm to (123.0, 67.9)
Routing:
- net +3.3V: track 0.00 -> 268.7 mm, vias 0 -> 4
- net +5V: track 0.00 -> 149.5 mm, vias 0 -> 4
- net /ID0: track 0.00 -> 142.2 mm, vias 0 -> 4
- net /EN: track 0.00 -> 132.7 mm, vias 0 -> 4
- net /HVBAT: track 0.00 -> 127.3 mm, vias 0 -> 2
- net Net-(U1-SENSOR_VP): track 0.00 -> 105.9 mm, vias 0 -> 2
- net Net-(D4-K): track 0.00 -> 96.5 mm, vias 0 -> 2
- net /DTR: track 0.00 -> 78.1 mm, vias 0 -> 3
- net /GPIO23: track 0.00 -> 62.2 mm, vias 0 -> 1
- net Net-(U5-PROG): track 0.00 -> 60.0 mm, vias 0 -> 2
- net Net-(Q3-G): track 0.00 -> 59.1 mm, vias 0 -> 2
- net /VRx: track 0.00 -> 56.2 mm
- net /GPIO18: track 0.00 -> 55.5 mm, vias 0 -> 1
- net /GPIO5: track 0.00 -> 54.1 mm, vias 0 -> 1
- net /GPIO15: track 0.00 -> 47.9 mm, vias 0 -> 1
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
Commit message: docu
Routing:
- net GND: track 43.9 -> 56.1 mm, vias 6 -> 8
