File: kicad/supply.kicad_sch (KiCad schematic)
At the start: 25 parts, among them J2 Conn_01x02, P1 USB_C_Plug_USB2.0, U5 TP4056-42-ESOP8, U6 USBLC6-2P6, U7 U8205A, U8 DW01A, U9 AMS1117-3.3

Commit message: init
Parts:
- U10: value ~ -> Switch
Changed lines of the file:
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@@
 			)
 		)
-		(property "Value" "~"
+		(property "Value" "Switch"
 			(at 190.5 135.89 0)
 			(effects

Commit message: init
Parts:
- R12: value 1.2K -> 2K
- R14: value R -> 10K
Changed lines of the file:
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@@
 			)
 		)
-		(property "Value" "1.2K"
+		(property "Value" "2K"
 			(at 121.92 143.5099 0)
 			(effects
@@
 			)
 		)
-		(property "Value" "R"
+		(property "Value" "10K"
 			(at 142.24 119.3799 0)
 			(effects

Commit message: init
Parts:
- removed R14: 10K, Resistor_SMD:R_1206_3216Metric, symbol Device:R
- removed R15: R, Resistor_SMD:R_1206_3216Metric, symbol Device:R
Connections:
- net GND: now also U5.1 (TEMP); no longer U5.9 (EPAD)
- no-connect marks 5 -> 6

Commit message: init
Connections:
- net at U7.2 (D1): now also U7.5 (D2)
- no-connect marks 6 -> 4
Changed lines of the file:
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@@
 	(paper "A4")
 	(rectangle
-		(start 55.88 91.44)
+		(start 55.88 88.9)
 		(end 205.74 160.02)
 		(stroke
@@
 	(text "Charger"
 		(exclude_from_sim no)
-		(at 59.69 90.17 0)
+		(at 59.436 87.884 0)
 		(effects
 			(font
@@
 	)
 	(no_connect
-		(at 163.83 133.35)
-	)
-	(no_connect
 		(at 92.71 36.83)
 	)
-	(no_connect
-		(at 163.83 148.59)
-	)
 	(wire
 		(pts
@@
 	(wire
 		(pts
-			(xy 66.04 95.25) (xy 76.2 95.25)
-		)
-		(stroke
-			(width 0)
-			(type default)
-		)
-	)
-	(wire
-		(pts
 			(xy 106.68 49.53) (xy 106.68 53.34)
 		)
@@
 	(wire
 		(pts
+			(xy 66.04 92.71) (xy 66.04 95.25)
+		)
+		(stroke
+			(width 0)
+			(type default)
+		)
+	)
+	(wire
+		(pts
 			(xy 130.81 143.51) (xy 130.81 148.59)
 		)
@@
 	(wire
 		(pts
+			(xy 172.72 132.08) (xy 172.72 152.4)
+		)
+		(stroke
+			(width 0)
+			(type default)
+		)
+	)
+	(wire
+		(pts
 			(xy 81.28 116.84) (xy 81.28 121.92)
 		)
@@
 	(wire
 		(pts
-			(xy 165.1 129.54) (xy 165.1 132.08)
+			(xy 165.1 129.54) (xy 165.1 130.81)
 		)
 		(stroke
@@
 	(wire
 		(pts
+			(xy 163.83 152.4) (xy 163.83 148.59)
+		)
+		(stroke
+			(width 0)
+			(type default)
+		)
+	)
+	(wire
+		(pts
 			(xy 69.85 67.31) (xy 69.85 69.85)
 		)
@@
 	(wire
 		(pts
-			(xy 167.64 132.08) (xy 167.64 133.35)
+			(xy 167.64 130.81) (xy 167.64 133.35)
 		)
 		(stroke
@@
 	(wire
 		(pts
-			(xy 165.1 132.08) (xy 167.64 132.08)
+			(xy 165.1 130.81) (xy 167.64 130.81)
 		)
 		(stroke
@@
 	(wire
 		(pts
+			(xy 172.72 152.4) (xy 163.83 152.4)
+		)
+		(stroke
+			(width 0)
+			(type default)
+		)
+	)
+	(wire
+		(pts
 			(xy 184.15 104.14) (xy 184.15 109.22)
 		)
@@
 		(pts
 			(xy 104.14 101.6) (xy 104.14 105.41)
+		)
+		(stroke
+			(width 0)
+			(type default)
+		)
+	)
+	(wire
+		(pts
+			(xy 163.83 132.08) (xy 163.83 133.35)
+		)
+		(stroke
+			(width 0)
+			(type default)
+		)
+	)
+	(wire
+		(pts
+			(xy 163.83 132.08) (xy 172.72 132.08)
 		)
 		(stroke
@@
 	(symbol
 		(lib_id "power:GND")
-		(at 76.2 95.25 90)
+		(at 66.04 92.71 180)
 		(unit 1)
 		(exclude_from_sim no)
@@
 		(dnp no)
 		(property "Reference" "#PWR022"
-			(at 82.55 95.25 0)
+			(at 66.04 86.36 0)
 			(effects
 				(font
@@
 		)
 		(property "Value" "GND"
-			(at 78.994 96.52 90)
+			(at 68.834 90.678 0)
 			(effects
 				(font
@@
 		)
 		(property "Footprint" ""
-			(at 76.2 95.25 0)
+			(at 66.04 92.71 0)
 			(effects
 				(font
@@
 		)
 		(property "Datasheet" ""
-			(at 76.2 95.25 0)
+			(at 66.04 92.71 0)
 			(effects
 				(font
@@
 		)
 		(property "Description" "Power symbol creates a global label with name \"GND\" , ground"
-			(at 76.2 95.25 0)
-			(effects
-				(font
+			(at 66.04 92.71 0)
+			(effects
+				(font

Commit message: init
Parts:
- removed J2: Conn_01x02, Connector_JST:JST_PH_B2B-PH-K_1x02_P2.00mm_Vertical, symbol Connector_Generic:Conn_01x02
- added U11: Battary, PCM_yvolodym:NCR18650B, symbol PCM_yvolodym:NCR18650B
Connections:
- net +3.3V: now also U11.1
- net at U10.2: now also U11.2
Changed lines of the file:
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@@
+	(wire
+		(pts
+			(xy 195.58 132.08) (xy 195.58 139.7)
+		)
+		(stroke
+			(width 0)
+			(type default)
+		)
+	)
 	(wire
 		(pts
@@
 		(pts
 			(xy 114.3 29.21) (xy 127 29.21)
-		)
-		(stroke
-			(width 0)
-			(type default)
-		)
-	)
-	(wire
-		(pts
-			(xy 195.58 128.27) (xy 195.58 139.7)
 		)
 		(stroke
@@
 	)
 	(symbol
+		(lib_id "PCM_yvolodym:NCR18650B")
+		(at 195.58 129.54 90)
+		(unit 1)
+		(exclude_from_sim no)
+		(in_bom yes)
+		(on_board yes)
+		(dnp no)
+		(property "Reference" "U11"
+			(at 201.422 125.476 90)
+			(effects
+				(font
+					(size 1.27 1.27)
+				)
+				(justify left)
+			)
+		)
+		(property "Value" "Battary"
+			(at 203.454 131.826 90)
+			(effects
+				(font
+					(size 1.27 1.27)
+				)
+				(justify left)
+			)
+		)
+		(property "Footprint" "PCM_yvolodym:NCR18650B"
+			(at 195.58 129.54 0)
+			(effects
+				(font
+					(size 1.27 1.27)
+				)
+				(hide yes)
+			)
+		)
+		(property "Datasheet" ""
+			(at 195.58 129.54 0)
+			(effects
+				(font
+					(size 1.27 1.27)
+				)
+				(hide yes)
+			)
+		)
+		(property "Description" ""
+			(at 195.58 129.54 0)
+			(effects
+				(font
+					(size 1.27 1.27)
+				)
+				(hide yes)
+			)
+		)
+		(pin "1"
+		)
+		(pin "2"
+		)
+		(instances
+			(project ""
+				(path "/1b61a099-fa01-45c5-bfa6-c1f023697108/13eaefed-e598-4605-b03d-de27b94da232"
+					(reference "U11")
+					(unit 1)
+				)
+			)
+		)
+	)
+	(symbol
 		(lib_id "power:GND")
 		(at 187.96 62.23 0)
@@
 				(path "/1b61a099-fa01-45c5-bfa6-c1f023697108/13eaefed-e598-4605-b03d-de27b94da232"
 					(reference "#PWR031")
-					(unit 1)
-				)
-			)
-		)
-	)
-	(symbol
-		(lib_id "Connector_Generic:Conn_01x02")
-		(at 200.66 125.73 0)
-		(unit 1)
-		(exclude_from_sim no)
-		(in_bom yes)
-		(on_board yes)
-		(dnp no)
-		(fields_autoplaced yes)
-		(property "Reference" "J2"
-			(at 203.2 125.7299 0)
-			(effects
-				(font
-					(size 1.27 1.27)
-				)
-				(justify left)
-			)
-		)
-		(property "Value" "Conn_01x02"
-			(at 203.2 128.2699 0)
-			(effects
-				(font
-					(size 1.27 1.27)
-				)
-				(justify left)
-			)
-		)
-		(property "Footprint" "Connector_JST:JST_PH_B2B-PH-K_1x02_P2.00mm_Vertical"
-			(at 200.66 125.73 0)
-			(effects
-				(font
-					(size 1.27 1.27)
-				)
-				(hide yes)
-			)
-		)
-		(property "Datasheet" "~"
-			(at 200.66 125.73 0)
-			(effects
-				(font
-					(size 1.27 1.27)
-				)
-				(hide yes)
-			)
-		)
-		(property "Description" "Generic connector, single row, 01x02, script generated (kicad-library-utils/schlib/autogen/connector/)"
-			(at 200.66 125.73 0)
-			(effects
-				(font
-					(size 1.27 1.27)
-				)
-				(hide yes)
-			)
-		)
-		(property "Sim.Device" ""
-			(at 200.66 125.73 0)
-			(effects
-				(font
-					(size 1.27 1.27)
-				)
-				(hide yes)
-			)
-		)
-		(property "Sim.Type" ""
-			(at 200.66 125.73 0)
-			(effects
-				(font
-					(size 1.27 1.27)
-				)
-				(hide yes)
-			)
-		)
-		(pin "2"
-		)
-		(pin "1"
-		)
-		(instances
-			(project "esp32-controller"
-				(path "/1b61a099-fa01-45c5-bfa6-c1f023697108/13eaefed-e598-4605-b03d-de27b94da232"
-					(reference "J2")
 					(unit 1)
 				)
@@
 		(on_board yes)
 		(dnp no)
-		(fields_autoplaced yes)
 		(property "Reference" "U10"
-			(at 190.5 133.35 0)
+			(at 194.31 143.002 0)
 			(effects
 				(font
@@
 		)
 		(property "Value" "Switch"
-			(at 190.5 135.89 0)
-			(effects
-				(font
+			(at 195.326 145.542 0)
+			(effects
+				(font

Commit message: init
Parts:
- D5: value LED -> BLAU
Changed lines of the file:
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@@
 			)
 		)
-		(property "Value" "LED"
+		(property "Value" "BLAU"
 			(at 143.51 51.1174 90)
 			(effects

Commit message: init
Parts:
- removed D3: GREEN, Diode_SMD:D_0603_1608Metric, symbol Device:LED
- removed R10: 1K, Resistor_SMD:R_1206_3216Metric, symbol Device:R
- renumbered D4 to D3, D5 to D4, R11 to R10, R12 to R11, R13 to R12, R16 to R13, R17 to R14
Connections:
- net GND: now also U5.6 (~{STDBY})
Other:
- moved on the sheet: C3

Commit message: GA install
Parts:
- added R15, R16: 5.1k, Resistor_SMD:R_0402_1005Metric, symbol Device:R
- U11: value Battary -> Battery
Connections:
- net +5V: now also U5.1 (TEMP)
- net GND: now also U5.9 (EPAD), R15.2, R16.2; no longer U5.1 (TEMP)
- net at P1.A5 (CC): now also R15.1
- net at P1.B5 (VCONN): now also R16.1
- no-connect marks 4 -> 1
Other:
- moved on the sheet: U6
