File: kicad/supply.kicad_sch (KiCad schematic)
At the start: 27 parts, among them P1 USB_C_Plug_USB2.0, Q3 SI2305, U10 Battery, U11 AP2112K-3.3, U12 LTC4412, U5 TP4056-42-ESOP8, U6 USBLC6-2P6, U7 U8205A, U8 DW01A, U9 Switch

Commit message: init
Parts:
- removed Q3: SI2305, Package_TO_SOT_SMD:SOT-23, symbol Device:Q_PMOS
- added Q3: Si2319CDS, Package_TO_SOT_SMD:SOT-23, symbol Transistor_FET:Si2319CDS
Connections:
- net GND: now also U12.3 (CTL)
- net Q1_GATE: now also Q3.1 (G)
- net VBAT: no longer U12.3 (CTL)
- net VPWR: now also Q3.3 (D)
- net at D6.1 (K): now also Q3.2 (S)
Changed lines of the file:
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@@
 	)
 	(junction
-		(at 241.3 95.25)
-		(diameter 0)
-		(color 0 0 0 0)
-	)
-	(junction
 		(at 118.11 36.83)
 		(diameter 0)
@@
 	(wire
 		(pts
-			(xy 242.57 90.17) (xy 241.3 90.17)
-		)
-		(stroke
-			(width 0)
-			(type default)
-		)
-	)
-	(wire
-		(pts
 			(xy 196.85 26.67) (xy 196.85 29.21)
 		)
@@
 	(wire
 		(pts
-			(xy 241.3 95.25) (xy 234.95 95.25)
+			(xy 234.95 95.25) (xy 242.57 95.25)
 		)
 		(stroke
@@
 	(wire
 		(pts
-			(xy 241.3 90.17) (xy 241.3 95.25)
-		)
-		(stroke
-			(width 0)
-			(type default)
-		)
-	)
-	(wire
-		(pts
 			(xy 149.86 48.26) (xy 149.86 59.69)
 		)
@@
 	(wire
 		(pts
-			(xy 242.57 95.25) (xy 241.3 95.25)
-		)
-		(stroke
-			(width 0)
-			(type default)
-		)
-	)
-	(wire
-		(pts
 			(xy 223.52 26.67) (xy 223.52 29.21)
 		)
@@
 	(wire
 		(pts
-			(xy 162.56 45.72) (xy 166.37 45.72)
+			(xy 163.83 45.72) (xy 166.37 45.72)
 		)
 		(stroke
@@
 	(wire
 		(pts
+			(xy 234.95 90.17) (xy 242.57 90.17)
+		)
+		(stroke
+			(width 0)
+			(type default)
+		)
+	)
+	(wire
+		(pts
 			(xy 223.52 48.26) (xy 223.52 59.69)
 		)
@@
 	)
 	(label "VBAT"
-		(at 162.56 45.72 180)
+		(at 234.95 90.17 0)
 		(effects
 			(font
 				(size 1.27 1.27)
 			)
-			(justify right)
+			(justify left bottom)
 		)
 	)
 	(label "VBAT"
-		(at 234.95 95.25 0)
+		(at 163.83 45.72 180)
 		(effects
 			(font
 				(size 1.27 1.27)
 			)
-			(justify left bottom)
+			(justify right)
 		)
 	)
@@
 		(dnp no)
 		(fields_autoplaced yes)
-		(property "Reference" "#PWR034"
+		(property "Reference" "#PWR035"
 			(at 252.73 113.03 0)
 			(effects
@@
 			(project "esp32-controller"
 				(path "/1b61a099-fa01-45c5-bfa6-c1f023697108/13eaefed-e598-4605-b03d-de27b94da232"
-					(reference "#PWR034")
+					(reference "#PWR035")
 					(unit 1)
 				)
@@
 	)
 	(symbol
-		(lib_id "Device:Q_PMOS")
-		(at 181.61 43.18 270)
-		(unit 1)
-		(exclude_from_sim no)
-		(in_bom yes)
-		(on_board yes)
-		(dnp no)
-		(property "Reference" "Q3"
-			(at 182.626 40.64 90)
-			(effects
-				(font
-					(size 1.27 1.27)
-				)
-				(justify left)
-			)
-		)
-		(property "Value" "SI2305"
-			(at 182.626 38.354 90)
-			(effects
-				(font
-					(size 1.27 1.27)
-				)
-				(justify left)
-			)
-		)
-		(property "Footprint" "Package_TO_SOT_SMD:SOT-23"
-			(at 181.61 43.18 0)
-			(effects
-				(font
-					(size 1.27 1.27)
-				)
-				(hide yes)
-			)
-		)
-		(property "Datasheet" "~"
-			(at 181.61 43.18 0)
-			(effects
-				(font
-					(size 1.27 1.27)
-				)
-				(hide yes)
-			)
-		)
-		(property "Description" "P-MOSFET transistor"
-			(at 181.61 43.18 0)
-			(effects
-				(font
-					(size 1.27 1.27)
-				)
-				(hide yes)
-			)
-		)
-		(pin "G"
-		)
-		(pin "S"
-		)
-		(pin "D"
-		)
-		(instances
-			(project "esp32-controller"
-				(path "/1b61a099-fa01-45c5-bfa6-c1f023697108/13eaefed-e598-4605-b03d-de27b94da232"
-					(reference "Q3")
-					(unit 1)
-				)
-			)
-		)
-	)
-	(symbol
 		(lib_id "Device:C")
 		(at 246.38 41.91 180)
@@
 		(dnp no)
 		(fields_autoplaced yes)
-		(property "Reference" "#PWR033"
+		(property "Reference" "#PWR034"
 			(at 246.38 54.61 0)
 			(effects
@@
 			(project "esp32-controller"
 				(path "/1b61a099-fa01-45c5-bfa6-c1f023697108/13eaefed-e598-4605-b03d-de27b94da232"
-					(reference "#PWR033")
+					(reference "#PWR034")
 					(unit 1)
 				)
@@
 	)
 	(symbol
+		(lib_id "Transistor_FET:Si2319CDS")
+		(at 181.61 43.18 270)
+		(unit 1)
+		(exclude_from_sim no)
+		(in_bom yes)
+		(on_board yes)
+		(dnp no)
+		(fields_autoplaced yes)
+		(property "Reference" "Q3"
+			(at 181.61 49.53 90)
+			(effects
+				(font
+					(size 1.27 1.27)
+				)
+			)
+		)
+		(property "Value" "Si2319CDS"
+			(at 181.61 52.07 90)
+			(effects
+				(font
+					(size 1.27 1.27)
+				)
+			)
+		)
+		(property "Footprint" "Package_TO_SOT_SMD:SOT-23"
+			(at 179.705 48.26 0)
+			(effects
+				(font
+					(size 1.27 1.27)
+					(italic yes)
+				)
+				(justify left)
+				(hide yes)
+			)
+		)
+		(property "Datasheet" "http://www.vishay.com/docs/66709/si2319cd.pdf"
+			(at 177.8 48.26 0)
+			(effects
+				(font
+					(size 1.27 1.27)
+				)
+				(justify left)
+				(hide yes)
+			)
+		)
+		(property "Description" "-4.4A Id, -40V Vds, P-Channel MOSFET, SOT-23"
+			(at 181.61 43.18 0)
+			(effects
+				(font
+					(size 1.27 1.27)
+				)
+				(hide yes)
+			)
+		)
+		(pin "1"
+		)
+		(pin "2"
+		)
+		(pin "3"
+		)
+		(instances
+			(project "esp32-controller"
+				(path "/1b61a099-fa01-45c5-bfa6-c1f023697108/13eaefed-e598-4605-b03d-de27b94da232"
+					(reference "Q3")
+					(unit 1)
+				)
+			)
+		)
+	)
+	(symbol
 		(lib_id "Device:C")
 		(at 81.28 99.06 180)
@@
 	)
 	(symbol
+		(lib_id "power:GND")
+		(at 234.95 95.25 0)
+		(unit 1)
+		(exclude_from_sim no)
+		(in_bom yes)
+		(on_board yes)
+		(dnp no)
+		(fields_autoplaced yes)
+		(property "Reference" "#PWR032"
+			(at 234.95 101.6 0)
+			(effects
+				(font
+					(size 1.27 1.27)
+				)
+				(hide yes)
+			)
+		)
+		(property "Value" "GND"
+			(at 234.95 100.965 0)
+			(effects
+				(font
+					(size 1.27 1.27)
+				)
+			)
+		)
+		(property "Footprint" ""
+			(at 234.95 95.25 0)
+			(effects
+				(font
+					(size 1.27 1.27)
+				)
+				(hide yes)
+			)
+		)
+		(property "Datasheet" ""
+			(at 234.95 95.25 0)
+			(effects
+				(font
+					(size 1.27 1.27)
+				)
+				(hide yes)
+			)
+		)
+		(property "Description" "Power symbol creates a global label with name \"GND\" , ground"
+			(at 234.95 95.25 0)
+			(effects
+				(font
+					(size 1.27 1.27)
+				)
+				(hide yes)
+			)
+		)
+		(pin "1"
+		)
+		(instances
+			(project "esp32-controller"
+				(path "/1b61a099-fa01-45c5-bfa6-c1f023697108/13eaefed-e598-4605-b03d-de27b94da232"
+					(reference "#PWR032")
+					(unit 1)
+				)
+			)
+		)
+	)
+	(symbol
 		(lib_id "Power_Protection:USBLC6-2P6")
 		(at 118.11 44.45 0)
@@
 		(dnp no)
 		(fields_autoplaced yes)
-		(property "Reference" "#PWR032"
+		(property "Reference" "#PWR033"
 			(at 246.38 40.64 0)
 			(effects
@@
 			(project "esp32-controller"
 				(path "/1b61a099-fa01-45c5-bfa6-c1f023697108/13eaefed-e598-4605-b03d-de27b94da232"
-					(reference "#PWR032")
+					(reference "#PWR033")
 					(unit 1)
 				)

Commit message: docu
Connections:
- net VBAT renamed HVBAT
Changed lines of the file:
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@@
+	)
+	(junction
+		(at 130.81 109.22)
+		(diameter 0)
+		(color 0 0 0 0)
 	)
 	(junction
@@
 		(pts
 			(xy 104.14 105.41) (xy 90.17 105.41)
+		)
+		(stroke
+			(width 0)
+			(type default)
+		)
+	)
+	(wire
+		(pts
+			(xy 130.81 105.41) (xy 130.81 109.22)
 		)
 		(stroke
@@
 		)
 	)
+	(hierarchical_label "HVBAT"
+		(shape input)
+		(at 130.81 105.41 90)
+		(effects
+			(font
+				(size 1.27 1.27)
+			)
+			(justify left)
+		)
+	)

Commit message: docu
Parts:
- C6: value 100pF -> 100nF
Changed lines of the file:
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@@
 			)
 		)
-		(property "Value" "100pF"
+		(property "Value" "100nF"
 			(at 188.468 131.572 0)
 			(effects

Commit message: docu
Parts:
- removed D6: SS14, Diode_SMD:D_SMA, symbol Diode:SS14
- renumbered C3 to C4, C4 to C5, C5 to C6, C6 to C7, C7 to C8, C8 to C9, R10 to R12, R11 to R13, R12 to R14, R13 to R15, R14 to R16, R15 to R17, R16 to R18
Connections:
- net HVBAT: now also Q3.3 (D)
- net VPWR: now also Q3.2 (S); no longer Q3.3 (D)
Other:
- moved on the sheet: Q3
