File: kicad/supply.kicad_sch (KiCad schematic)
At the start: 26 parts, among them P1 USB_C_Plug_USB2.0, Q3 Si2319CDS, U10 Battery, U11 AP2112K-3.3, U12 LTC4412, U5 TP4056-42-ESOP8, U6 USBLC6-2P6, U7 U8205A, U8 DW01A, U9 Switch

Commit message: docu
Parts:
- R16: value 2K -> 470
Connections:
- net +3.3V: now also R16.1
- net +5V: no longer R16.1
Other:
- moved on the sheet: C6, C7, C8, C9, D4, D5, Q3, R16, R17, R18, U10, U11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

Commit message: docu
Parts:
- D3: value RED -> BATT
- D4: value BLAU -> NET
Changed lines of the file:
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@@
 			)
 		)
-		(property "Value" "RED"
+		(property "Value" "BATT"
 			(at 85.09 115.8874 90)
 			(effects
@@
 			)
 		)
-		(property "Value" "BLAU"
+		(property "Value" "NET"
 			(at 202.692 55.88 90)
 			(effects

Commit message: docu
Parts:
- D3: value BATT -> LED_RED
- D4: value NET -> LED_GREEN
Changed lines of the file:
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@@
 			)
 		)
-		(property "Value" "BATT"
+		(property "Value" "LED_RED"
 			(at 85.09 115.8874 90)
 			(effects
@@
 			)
 		)
-		(property "Value" "NET"
+		(property "Value" "LED_GREEN"
 			(at 202.692 55.88 90)
 			(effects

Commit message: init
Parts:
- D3, D4: footprint Diode_SMD:D_0603_1608Metric -> LED_THT:LED_D2.0mm_W4.8mm_H2.5mm_FlatTop
Changed lines of the file:
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@@
 		(on_board yes)
 		(dnp no)
-		(fields_autoplaced yes)
 		(property "Reference" "D3"
-			(at 85.09 113.3474 90)
+			(at 75.692 109.728 90)
 			(effects
 				(font
@@
 		)
 		(property "Value" "LED_RED"
-			(at 85.09 115.8874 90)
+			(at 70.358 112.522 90)
 			(effects
 				(font
@@
 			)
 		)
-		(property "Footprint" "Diode_SMD:D_0603_1608Metric"
+		(property "Footprint" "LED_THT:LED_D2.0mm_W4.8mm_H2.5mm_FlatTop"
 			(at 81.28 113.03 0)
 			(effects
@@
 		)
 		(property "Value" "LED_GREEN"
-			(at 202.692 55.88 90)
+			(at 198.374 50.8 90)
 			(effects
 				(font
@@
 			)
 		)
-		(property "Footprint" "Diode_SMD:D_0603_1608Metric"
+		(property "Footprint" "LED_THT:LED_D2.0mm_W4.8mm_H2.5mm_FlatTop"
 			(at 209.55 54.61 0)
 			(effects

Commit message: docu
Parts:
- renumbered D5 to D4, D4 to D5, R17 to R16, R18 to R17, R16 to R18, U9 to U10, U10 to U11, U11 to U12, U12 to U9
Changed lines of the file:
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@@
 		(on_board yes)
 		(dnp no)
-		(property "Reference" "U10"
+		(property "Reference" "U11"
 			(at 193.802 125.476 90)
 			(effects
@@
 			(project "esp32-controller"
 				(path "/1b61a099-fa01-45c5-bfa6-c1f023697108/13eaefed-e598-4605-b03d-de27b94da232"
-					(reference "U10")
+					(reference "U11")
 					(unit 1)
 				)
@@
 		(on_board yes)
 		(dnp no)
-		(property "Reference" "U9"
+		(property "Reference" "U10"
 			(at 186.69 143.002 0)
 			(effects
@@
 			(project "esp32-controller"
 				(path "/1b61a099-fa01-45c5-bfa6-c1f023697108/13eaefed-e598-4605-b03d-de27b94da232"
-					(reference "U9")
+					(reference "U10")
 					(unit 1)
 				)
@@
 		(dnp no)
 		(fields_autoplaced yes)
-		(property "Reference" "U11"
+		(property "Reference" "U12"
 			(at 196.85 22.86 0)
 			(effects
@@
 			(project "esp32-controller"
 				(path "/1b61a099-fa01-45c5-bfa6-c1f023697108/13eaefed-e598-4605-b03d-de27b94da232"
-					(reference "U11")
+					(reference "U12")
 					(unit 1)
 				)
@@
 		(on_board yes)
 		(dnp no)
-		(property "Reference" "D4"
+		(property "Reference" "D5"
 			(at 204.978 53.34 90)
 			(effects
@@
 			(project "esp32-controller"
 				(path "/1b61a099-fa01-45c5-bfa6-c1f023697108/13eaefed-e598-4605-b03d-de27b94da232"
-					(reference "D4")
+					(reference "D5")
 					(unit 1)
 				)
@@
 		(dnp no)
 		(fields_autoplaced yes)
-		(property "Reference" "R18"
+		(property "Reference" "R17"
 			(at 181.61 113.03 90)
 			(effects
@@
 			(project "esp32-controller"
 				(path "/1b61a099-fa01-45c5-bfa6-c1f023697108/13eaefed-e598-4605-b03d-de27b94da232"
-					(reference "R18")
+					(reference "R17")
 					(unit 1)
 				)
@@
 		(dnp no)
 		(fields_autoplaced yes)
-		(property "Reference" "R17"
+		(property "Reference" "R16"
 			(at 143.51 132.0799 0)
 			(effects
@@
 			(project "esp32-controller"
 				(path "/1b61a099-fa01-45c5-bfa6-c1f023697108/13eaefed-e598-4605-b03d-de27b94da232"
-					(reference "R17")
+					(reference "R16")
 					(unit 1)
 				)
@@
 		(dnp no)
 		(fields_autoplaced yes)
-		(property "Reference" "#FLG05"
+		(property "Reference" "#FLG02"
 			(at 83.185 -63.5 0)
 			(effects
@@
 			(project "esp32-controller"
 				(path "/1b61a099-fa01-45c5-bfa6-c1f023697108/13eaefed-e598-4605-b03d-de27b94da232"
-					(reference "#FLG05")
+					(reference "#FLG02")
 					(unit 1)
 				)
@@
 		(dnp no)
 		(fields_autoplaced yes)
-		(property "Reference" "#FLG04"
+		(property "Reference" "#FLG05"
 			(at 105.41 22.225 0)
 			(effects
@@
 			(project "esp32-controller"
 				(path "/1b61a099-fa01-45c5-bfa6-c1f023697108/13eaefed-e598-4605-b03d-de27b94da232"
-					(reference "#FLG04")
+					(reference "#FLG05")
 					(unit 1)
 				)
@@
 		(on_board yes)
 		(dnp no)
-		(property "Reference" "U12"
+		(property "Reference" "U9"
 			(at 154.432 70.104 0)
 			(effects
@@
 			(project "esp32-controller"
 				(path "/1b61a099-fa01-45c5-bfa6-c1f023697108/13eaefed-e598-4605-b03d-de27b94da232"
-					(reference "U12")
+					(reference "U9")
 					(unit 1)
 				)
@@
 		(dnp no)
 		(fields_autoplaced yes)
-		(property "Reference" "#PWR035"
+		(property "Reference" "#PWR034"
 			(at 243.84 54.61 0)
 			(effects
@@
 			(project "esp32-controller"
 				(path "/1b61a099-fa01-45c5-bfa6-c1f023697108/13eaefed-e598-4605-b03d-de27b94da232"
-					(reference "#PWR035")
+					(reference "#PWR034")
 					(unit 1)
 				)
@@
 		(on_board yes)
 		(dnp no)
-		(property "Reference" "R16"
+		(property "Reference" "R18"
 			(at 203.708 41.91 0)
 			(effects
@@
 			(project "esp32-controller"
 				(path "/1b61a099-fa01-45c5-bfa6-c1f023697108/13eaefed-e598-4605-b03d-de27b94da232"
-					(reference "R16")
+					(reference "R18")
 					(unit 1)
 				)
@@
 		(dnp no)
 		(fields_autoplaced yes)
-		(property "Reference" "#FLG03"
+		(property "Reference" "#FLG04"
 			(at 173.99 153.035 0)
 			(effects
@@
 			(project "esp32-controller"
 				(path "/1b61a099-fa01-45c5-bfa6-c1f023697108/13eaefed-e598-4605-b03d-de27b94da232"
-					(reference "#FLG03")
+					(reference "#FLG04")
 					(unit 1)
 				)
@@
 		(on_board yes)
 		(dnp no)
-		(property "Reference" "#FLG02"
+		(property "Reference" "#FLG03"
 			(at 173.99 113.665 0)
 			(effects
@@
 			(project "esp32-controller"
 				(path "/1b61a099-fa01-45c5-bfa6-c1f023697108/13eaefed-e598-4605-b03d-de27b94da232"
-					(reference "#FLG02")
+					(reference "#FLG03")
 					(unit 1)
 				)
@@
 		(dnp no)
 		(fields_autoplaced yes)
-		(property "Reference" "#PWR034"
+		(property "Reference" "#PWR033"
 			(at 243.84 40.64 0)
 			(effects
@@
 			(project "esp32-controller"
 				(path "/1b61a099-fa01-45c5-bfa6-c1f023697108/13eaefed-e598-4605-b03d-de27b94da232"
-					(reference "#PWR034")
+					(reference "#PWR033")
 					(unit 1)
 				)
@@
 		(dnp no)
 		(fields_autoplaced yes)
-		(property "Reference" "D5"
+		(property "Reference" "D4"
 			(at 151.4475 22.86 0)
 			(effects
@@
 			(project "esp32-controller"
 				(path "/1b61a099-fa01-45c5-bfa6-c1f023697108/13eaefed-e598-4605-b03d-de27b94da232"
-					(reference "D5")
+					(reference "D4")
 					(unit 1)
 				)

Commit message: docu
Parts:
- U10: footprint PCM_yvolodym:Switch -> Button_Switch_SMD:SW_SPDT_PCM12
Changed lines of the file:
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@@
 			)
 		)
-		(property "Footprint" "PCM_yvolodym:Switch"
+		(property "Footprint" "Button_Switch_SMD:SW_SPDT_PCM12"
 			(at 182.626 134.366 0)
 			(effects
